File: MES4_Carrier_EC/AuxPower.kicad_sch (KiCad schematic)
At the start: 36 parts, among them J14 IMU 9V, J15 SERVO 24V, J16 SCREEN 5V, J17 SERVO UART, SW2 SS12D10G5, U10 URB2409S-10WR3, U11 URB2405LD-20WR3

Commit message: Put relay coil feedback back on PA0-PA3 (MES4 GPIO standard)
All 14 module GPIOs now follow the MES4-CIF §2c table. The TCA9535 is
removed from the Relays 3-4 sheet and J1 fingers 43/45/47/49 drive the
relay 1-4 feedback dividers again. The winch relays are left undriven
(gate inputs no-connected, 100k pull-downs hold them off) until they
move to the TCA9535 + photoMOS design (HANDOFF.md step 2).

Removing U4 renumbers U5-U12 to U4-U11 and C15-C45 to C14-C44; the
README refs follow. Adds generator/checks.py (pin/pad, single-pin nets,
duplicate UUIDs, LCSC numbers), run by run.sh after ERC.

Co-Authored-By: Claude Opus 5.5 <noreply@anthropic.com>
Parts:
- removed C31: 10uF 50V, Capacitor_SMD:C_0805_2012Metric, symbol Device:C
- removed C33, C35, C37: 47uF 100V, Capacitor_SMD:CP_Elec_8x10, symbol Device:C_Polarized
- removed C34: 22uF 16V, Capacitor_SMD:C_0805_2012Metric, symbol Device:C
- removed C36: 100nF 50V, Capacitor_SMD:C_0603_1608Metric, symbol Device:C
- removed C42: 2.2uF, Capacitor_SMD:C_0402_1005Metric, symbol Device:C
- removed D23: H5VSD3B, Diode_SMD:D_SOD-323, symbol Device:D_TVS
- removed F11: 3A, Fuse:Fuse_2920_7451Metric, symbol Device:Polyfuse
- removed U10: URB2409S-10WR3, MES4-Carrier-EC:PWRM-TH_YLPTEC_URBXXXXS-10WR3, symbol MES4-Carrier-EC:URB2409S-10WR3
- removed U11: URB2405LD-20WR3, MES4-Carrier-EC:PWRM-TH_YLPTEC_URBXXXXLD-20WR3, symbol MES4-Carrier-EC:URB2405LD-20WR3
- added C30: 10uF 50V, Capacitor_SMD:C_0805_2012Metric, symbol Device:C
- added C31: 100uF 63V, Capacitor_SMD:CP_Elec_8x10, symbol Device:C_Polarized
- added C33: 22uF 16V, Capacitor_SMD:C_0805_2012Metric, symbol Device:C
- added C34, C36: 47uF 100V, Capacitor_SMD:CP_Elec_8x10, symbol Device:C_Polarized
- added C35: 100nF 50V, Capacitor_SMD:C_0603_1608Metric, symbol Device:C
- added C37: 22uF 25V, Capacitor_SMD:C_0805_2012Metric, symbol Device:C
- added C39: 100nF, Capacitor_SMD:C_0402_1005Metric, symbol Device:C
- added R44: 10k, Resistor_SMD:R_0402_1005Metric, symbol Device:R
- added U10: URB2405LD-20WR3, MES4-Carrier-EC:PWRM-TH_YLPTEC_URBXXXXLD-20WR3, symbol MES4-Carrier-EC:URB2405LD-20WR3
- added U9: URB2409S-10WR3, MES4-Carrier-EC:PWRM-TH_YLPTEC_URBXXXXS-10WR3, symbol MES4-Carrier-EC:URB2409S-10WR3
- C32: value 100uF 63V -> 47uF 100V; LCSC C48970912 -> C48935391
- C41: value 100nF -> 2.2uF; LCSC C1525 -> C12530
- D23: renamed from R44; value 10k -> H5VSD3B; footprint Resistor_SMD:R_0402_1005Metric -> Diode_SMD:D_SOD-323; symbol Device:R -> Device:D_TVS; LCSC C25744 -> C20615806
- F11: renamed from C39; value 22uF 25V -> 3A; footprint Capacitor_SMD:C_0805_2012Metric -> Fuse:Fuse_2920_7451Metric; symbol Device:C -> Device:Polyfuse; LCSC C45783 -> C22435908
Connections:
- net +24V_AUX: now also C30.1, C31.1, C34.1, U10.2 (+Vin), U9.2 (VIN)
- net +24V_SRV: now also C35.1, C36.1
- net +3V3_MOD: now also R44.1; no longer D23.1
- net +5V_SCR: now also C37.1, C39.1, U10.3 (+Vo); no longer C40.1
- net +5V_SRV: now also C40.1; no longer C41.1
- net +9V_IMU: now also C33.1, U9.6 (+Vo)
- net GND: now also D23.2 (A2), C33.2, C37.2, C39.2, U10.5 (GND), U9.7 (-Vo); no longer F11.2
- net GND_24V: now also C30.2, C31.2, C34.2, C35.2, C36.2, U10.1 (-Vin), U9.1 (GND)
- net SCR_SHIELD: now also C41.1
- net SRV_RX: now also D23.1 (A1)
- net SRV_UART_RX: now also R44.2; no longer D23.2
- net VBUS_SCR: now also F11.2
Other:
- note added: "L2 10 µH (same part as L1) + C30 / C31: a pi filter of its own for the IMU and screen converters, so the screen's 20 W converter neither loads nor disturbs the logic supply (L1, Power sheet). Load at 24 V: IMU ≤ 0.5 A + screen ≤ 0.95 A ≈ 1.45 A; L2 is rated 2.1 A (2.9 A saturation). Both converters are isolated: input side on GND_24V, output side on GND (same scheme as the logic DC/DC)."
- note added: "Same parts as the MES3.1-Carrier-LH "IMU Power Supply @ 9V": U9 YLPTEC URB2409S-10WR3 (9-36 V in, 9 V 1.11 A, 10 W isolated, short-circuit protected; MES3.1 U15), C32 47 µF / 100 V and C33 22 µF / 16 V (the datasheet's Cin / Cout), SW2 SS12D10G5 slide switch (MES3.1 U22, common = pin 2), J14 KF250NH 2-pin (MES3.1 CN10). CTRL open = on. SW2 is rated 0.5 A: check the IMU draws less (the converter g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"
- note added: "U10 YLPTEC URB2405LD-20WR3: 9-36 V in, 5 V 4 A, 20 W isolated, short-circuit protected, 2" x 1" DIP. CTRL and Trim open (on, 5.0 V). C34 47 µF (datasheet C1 47-100 µF), C37 / C38 22 µF (C2 / C3 10-22 µF). F11 3 A PTC (same part as the relay outputs) + D22 SMF6.0A, then J16: the MES4-Flasher's USB-C power-only receptacle, rated 5 V 3 A (3 A on VBUS; GND pins 1.25 A each). R48 / R47 10k Rp to 5 V o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"
- note removed: "L2 10 µH (same part as L1) + C31 / C32: a pi filter of its own for the IMU and screen converters, so the screen's 20 W converter neither loads nor disturbs the logic supply (L1, Power sheet). Load at 24 V: IMU ≤ 0.5 A + screen ≤ 0.95 A ≈ 1.45 A; L2 is rated 2.1 A (2.9 A saturation). Both converters are isolated: input side on GND_24V, output side on GND (same scheme as the logic DC/DC)."
- note removed: "Same parts as the MES3.1-Carrier-LH "IMU Power Supply @ 9V": U10 YLPTEC URB2409S-10WR3 (9-36 V in, 9 V 1.11 A, 10 W isolated, short-circuit protected; MES3.1 U15), C33 47 µF / 100 V and C34 22 µF / 16 V (the datasheet's Cin / Cout), SW2 SS12D10G5 slide switch (MES3.1 U22, common = pin 2), J14 KF250NH 2-pin (MES3.1 CN10). CTRL open = on. SW2 is rated 0.5 A: check the IMU draws less (the converter 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"
- note removed: "U11 YLPTEC URB2405LD-20WR3: 9-36 V in, 5 V 4 A, 20 W isolated, short-circuit protected, 2" x 1" DIP. CTRL and Trim open (on, 5.0 V). C35 47 µF (datasheet C1 47-100 µF), C38 / C39 22 µF (C2 / C3 10-22 µF). F11 3 A PTC (same part as the relay outputs) + D22 SMF6.0A, then J16: the MES4-Flasher's USB-C power-only receptacle, rated 5 V 3 A (3 A on VBUS; GND pins 1.25 A each). R48 / R47 10k Rp to 5 V o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"

Commit message: Drop relay coil feedback; winch on PA0/PA1, servo on USART2
User decision: free the four feedback pins instead of adding an I²C
expander. The Flasher template's 10k/15k/10 nF dividers are removed from
all relay channels and relay diagnosis is INA226-only. PA0/PA1 drive the
IM03GR winch relays again and PA2/PA3 carry the door servo UART
(USART2), so the SC16IS740 bridge, its crystal and caps, and the unused
TCA9535 code are removed. This deliberately differs from the MES4-CIF
§2c GPIO table; the GPIO map, root notes, README and HANDOFF say so.

189 parts, ERC clean, checks.py passes. README refs follow the
renumbering.

Co-Authored-By: Claude Opus 5.5 <noreply@anthropic.com>
Parts:
- removed C30: 10uF 50V, Capacitor_SMD:C_0805_2012Metric, symbol Device:C
- removed C31: 100uF 63V, Capacitor_SMD:CP_Elec_8x10, symbol Device:C_Polarized
- removed C33: 22uF 16V, Capacitor_SMD:C_0805_2012Metric, symbol Device:C
- removed C36: 47uF 100V, Capacitor_SMD:CP_Elec_8x10, symbol Device:C_Polarized
- removed C38: 22uF 25V, Capacitor_SMD:C_0805_2012Metric, symbol Device:C
- removed C39, C40: 100nF, Capacitor_SMD:C_0402_1005Metric, symbol Device:C
- removed C41: 2.2uF, Capacitor_SMD:C_0402_1005Metric, symbol Device:C
- removed F10: 1.1A, Fuse:Fuse_1206_3216Metric, symbol Device:Polyfuse
- removed R43: 2.2k, Resistor_SMD:R_0402_1005Metric, symbol Device:R
- removed R44, R47, R48: 10k, Resistor_SMD:R_0402_1005Metric, symbol Device:R
- removed R45, R46: 100Ω, Resistor_SMD:R_0402_1005Metric, symbol Device:R
- removed R49: 1M, Resistor_SMD:R_0603_1608Metric, symbol Device:R
- removed SW2: SS12D10G5, MES4-Carrier-EC:SW-TH_SHOU-HAN_SS12D10G4, symbol Switch:SW_SPDT
- added C26: 10uF 50V, Capacitor_SMD:C_0805_2012Metric, symbol Device:C
- added C27: 100uF 63V, Capacitor_SMD:CP_Elec_8x10, symbol Device:C_Polarized
- added C28, C30: 47uF 100V, Capacitor_SMD:CP_Elec_8x10, symbol Device:C_Polarized
- added C29: 22uF 16V, Capacitor_SMD:C_0805_2012Metric, symbol Device:C
- added C31: 100nF 50V, Capacitor_SMD:C_0603_1608Metric, symbol Device:C
- added C34: 22uF 25V, Capacitor_SMD:C_0805_2012Metric, symbol Device:C
- added C36: 100nF, Capacitor_SMD:C_0402_1005Metric, symbol Device:C
- added D24: H5VSD3B, Diode_SMD:D_SOD-323, symbol Device:D_TVS
- added J16: SCREEN 5V, MES4-Carrier-EC:USB-C_Receptacle_PowerOnly_6P_C456012, symbol Connector:USB_C_Receptacle_PowerOnly_6P
- added R35: 2.2k, Resistor_SMD:R_0402_1005Metric, symbol Device:R
- added R36, R39, R40: 10k, Resistor_SMD:R_0402_1005Metric, symbol Device:R
- added R37, R38: 100Ω, Resistor_SMD:R_0402_1005Metric, symbol Device:R
- added R41: 1M, Resistor_SMD:R_0603_1608Metric, symbol Device:R
- C33: renamed from J16; value SCREEN 5V -> 22uF 25V; footprint MES4-Carrier-EC:USB-C_Receptacle_PowerOnly_6P_C456012 -> Capacitor_SMD:C_0805_2012Metric; symbol Connector:USB_C_Receptacle_PowerOnly_6P -> Device:C; LCSC C456012 -> C45783
- C35: value 100nF 50V -> 100nF; footprint Capacitor_SMD:C_0603_1608Metric -> Capacitor_SMD:C_0402_1005Metric; LCSC C14663 -> C1525
- C37: value 22uF 25V -> 2.2uF; footprint Capacitor_SMD:C_0805_2012Metric -> Capacitor_SMD:C_0402_1005Metric; LCSC C45783 -> C12530
- F10: renamed from D24; value H5VSD3B -> 1.1A; footprint Diode_SMD:D_SOD-323 -> Fuse:Fuse_1206_3216Metric; symbol Device:D_TVS -> Device:Polyfuse; LCSC C20615806 -> C126818
- SW2: renamed from C34; value 47uF 100V -> SS12D10G5; footprint Capacitor_SMD:CP_Elec_8x10 -> MES4-Carrier-EC:SW-TH_SHOU-HAN_SS12D10G4; symbol Device:C_Polarized -> Switch:SW_SPDT; LCSC C48935391 -> C7431054
Connections:
- net +24V_AUX: now also C26.1, C27.1, C28.1, C30.1; no longer C32.1, SW2.1
- net +24V_SRV: now also C32.1, C31.1; no longer C35.1
- net +3V3_MOD: now also R36.1
- net +5V_SCR: now also C33.1, C35.1, F10.1, C34.1; no longer C37.1
- net +5V_SRV: now also F10.2, C36.1
- net +9V_IMU: now also SW2.2 (B), C29.1
- net GND: now also C33.2, C35.2, C29.2, C34.2, C36.2, D24.2 (A2), J16.A12 (GND), J16.B12 (GND), R41.2; no longer C33.A12 (GND), C33.B12 (GND), F10.2 (A2)
- net GND_24V: now also C26.2, C27.2, C28.2, C30.2, C31.2; no longer C35.2, SW2.2
- net IMU_9V: now also SW2.1 (A), R35.1
- net SCR_CC1: now also J16.A5 (CC1), R40.2; no longer C33.A5 (CC1)
- net SCR_CC2: now also J16.B5 (CC2), R39.2; no longer C33.B5 (CC2)
- net SCR_SHIELD: now also C37.1, J16.S1 (SHIELD), R41.1; no longer C33.S1 (SHIELD)
- net SRV_RX: now also R37.2
- net SRV_TX: now also D24.1 (A1), R38.2; no longer F10.1 (A1)
- net VBUS_SCR: now also J16.A9 (VBUS), J16.B9 (VBUS), R39.1, R40.1; no longer C33.A9 (VBUS), C33.B9 (VBUS)
- net at LED8.2 (A): now also R35.2
- new net PA2: R38.1
- new net PA3: R36.2, R37.1
Other:
- note added: "J15 SERVO 24V and J17 SERVO UART: same pinout as CN5 / CN13 on the MES2 Harvester, so its cables fit. The FE-URT-2 turns the UART into the Feetech half-duplex servo bus and passes the 24 V on to the servos. UART on module USART2: PA2 TX → pin 4, pin 3 → PA3 RX (5 V-tolerant). F9 3 A PTC on the servo 24 V. F10 1.1 A PTC on the FE-URT-2 5 V, fed from the screen converter so a servo-side short can't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"
- note added: "L2 10 µH (same part as L1) + C26 / C27: a pi filter of its own for the IMU and screen converters, so the screen's 20 W converter neither loads nor disturbs the logic supply (L1, Power sheet). Load at 24 V: IMU ≤ 0.5 A + screen ≤ 0.95 A ≈ 1.45 A; L2 is rated 2.1 A (2.9 A saturation). Both converters are isolated: input side on GND_24V, output side on GND (same scheme as the logic DC/DC)."
- note added: "Same parts as the MES3.1-Carrier-LH "IMU Power Supply @ 9V": U9 YLPTEC URB2409S-10WR3 (9-36 V in, 9 V 1.11 A, 10 W isolated, short-circuit protected; MES3.1 U15), C28 47 µF / 100 V and C29 22 µF / 16 V (the datasheet's Cin / Cout), SW2 SS12D10G5 slide switch (MES3.1 U22, common = pin 2), J14 KF250NH 2-pin (MES3.1 CN10). CTRL open = on. SW2 is rated 0.5 A: check the IMU draws less (the converter g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"
- note added: "U10 YLPTEC URB2405LD-20WR3: 9-36 V in, 5 V 4 A, 20 W isolated, short-circuit protected, 2" x 1" DIP. CTRL and Trim open (on, 5.0 V). C30 47 µF (datasheet C1 47-100 µF), C33 / C34 22 µF (C2 / C3 10-22 µF). F11 3 A PTC (same part as the relay outputs) + D22 SMF6.0A, then J16: the MES4-Flasher's USB-C power-only receptacle, rated 5 V 3 A (3 A on VBUS; GND pins 1.25 A each). R40 / R39 10k Rp to 5 V o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"
- note removed: "J15 SERVO 24V and J17 SERVO UART: same pinout as CN5 / CN13 on the MES2 Harvester, so its cables fit. The FE-URT-2 turns the UART into the Feetech half-duplex servo bus and passes the 24 V on to the servos. UART from the SC16IS740 I²C bridge (Winch sheet, 0x48): TX → pin 4, pin 3 → RX. F9 3 A PTC on the servo 24 V. F10 1.1 A PTC on the FE-URT-2 5 V, fed from the screen converter so a servo-side s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"
- note removed: "L2 10 µH (same part as L1) + C30 / C31: a pi filter of its own for the IMU and screen converters, so the screen's 20 W converter neither loads nor disturbs the logic supply (L1, Power sheet). Load at 24 V: IMU ≤ 0.5 A + screen ≤ 0.95 A ≈ 1.45 A; L2 is rated 2.1 A (2.9 A saturation). Both converters are isolated: input side on GND_24V, output side on GND (same scheme as the logic DC/DC)."
- note removed: "Same parts as the MES3.1-Carrier-LH "IMU Power Supply @ 9V": U9 YLPTEC URB2409S-10WR3 (9-36 V in, 9 V 1.11 A, 10 W isolated, short-circuit protected; MES3.1 U15), C32 47 µF / 100 V and C33 22 µF / 16 V (the datasheet's Cin / Cout), SW2 SS12D10G5 slide switch (MES3.1 U22, common = pin 2), J14 KF250NH 2-pin (MES3.1 CN10). CTRL open = on. SW2 is rated 0.5 A: check the IMU draws less (the converter g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"
- note removed: "U10 YLPTEC URB2405LD-20WR3: 9-36 V in, 5 V 4 A, 20 W isolated, short-circuit protected, 2" x 1" DIP. CTRL and Trim open (on, 5.0 V). C34 47 µF (datasheet C1 47-100 µF), C37 / C38 22 µF (C2 / C3 10-22 µF). F11 3 A PTC (same part as the relay outputs) + D22 SMF6.0A, then J16: the MES4-Flasher's USB-C power-only receptacle, rated 5 V 3 A (3 A on VBUS; GND pins 1.25 A each). R48 / R47 10k Rp to 5 V o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"
- moved on the sheet: F10

Commit message: Add module finger map page and FE-URT-2 3.3 V note
New page 11 (Pinout): a KiCad table of every MES4-MCU finger with its
STM32 port, function, what this carrier connects to it, the carrier
parts, the MES4-CIF §2c standard use and notes. It follows the MES4-MCU
U1 pin map style (colour-coded Function column, spanned finger-group
rows); the PA0-PA3 rows mark where this board differs from §2c. The
builder gains table() with per-cell fills and row spans, and cell text
resolves {tag} references.

The AuxPower servo note, README and HANDOFF now say to set the FE-URT-2
level switch to 3.3 V: at 5 V its TX exceeds PA3's limit while the
module is unpowered and back-feeds the 3V3 through the RX pull-up.

Co-Authored-By: Claude Opus 5.5 <noreply@anthropic.com>
Other:
- note added: "J15 SERVO 24V and J17 SERVO UART: same pinout as CN5 / CN13 on the MES2 Harvester, so its cables fit. The FE-URT-2 turns the UART into the Feetech half-duplex servo bus and passes the 24 V on to the servos. UART on module USART2: PA2 TX → pin 4, pin 3 → PA3 RX (5 V-tolerant). Set the FE-URT-2 level switch to 3.3 V (not 5 V): it only sets the UART levels, the servo 24 V is unchanged. At 5 V its TX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"
- note removed: "J15 SERVO 24V and J17 SERVO UART: same pinout as CN5 / CN13 on the MES2 Harvester, so its cables fit. The FE-URT-2 turns the UART into the Feetech half-duplex servo bus and passes the 24 V on to the servos. UART on module USART2: PA2 TX → pin 4, pin 3 → PA3 RX (5 V-tolerant). F9 3 A PTC on the servo 24 V. F10 1.1 A PTC on the FE-URT-2 5 V, fed from the screen converter so a servo-side short can't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"

Commit message: Isolate the 48 V winch side, add servo TX pull-up, tidy block diagram
Winch: J18 and the WINCH_* / ILK_* nets already touch only relay
contacts; they now form net class Winch_48V (0.6 mm clearance), and the
Winch sheet, README and HANDOFF state the isolation rules (>= 2 mm to
other copper, no GND pour under J18, no ESD to GND on J18).

Servo: R37 10k pull-up holds PA2 (TX) idle HIGH while the MCU is in
reset. AuxPower/Winch refs R37-R45 shift by one; README follows, and the
LED8 resistor ref is corrected to R35.

Block diagram: door servo block, winch and servo links from the module,
24 V routed so it never crosses a signal line, channel lines on an even
5.08 mm pitch.

Co-Authored-By: Claude Opus 5.5 <noreply@anthropic.com>
Parts:
- added R39: 100Ω, Resistor_SMD:R_0402_1005Metric, symbol Device:R
- R37: renamed from R38; value 100Ω -> 10k; LCSC C25076 -> C25744
- renumbered R37 to R38, R39 to R40, R40 to R41, R41 to R42
Connections:
- net +3V3_MOD: now also R37.1
- net PA2: now also R37.2, R39.1; no longer R37.1
- net SRV_TX: now also R39.2; no longer R37.2
Other:
- note added: "J15 SERVO 24V and J17 SERVO UART: same pinout as CN5 / CN13 on the MES2 Harvester, so its cables fit. The FE-URT-2 turns the UART into the Feetech half-duplex servo bus and passes the 24 V on to the servos. UART on module USART2: PA2 TX → pin 4, pin 3 → PA3 RX (5 V-tolerant). R36 / R37 10k pull-ups keep RX / TX idle HIGH (TX floats in reset). Set the FE-URT-2 level switch to 3.3 V (not 5 V): it o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"
- note added: "U10 YLPTEC URB2405LD-20WR3: 9-36 V in, 5 V 4 A, 20 W isolated, short-circuit protected, 2" x 1" DIP. CTRL and Trim open (on, 5.0 V). C30 47 µF (datasheet C1 47-100 µF), C33 / C34 22 µF (C2 / C3 10-22 µF). F11 3 A PTC (same part as the relay outputs) + D22 SMF6.0A, then J16: the MES4-Flasher's USB-C power-only receptacle, rated 5 V 3 A (3 A on VBUS; GND pins 1.25 A each). R41 / R40 10k Rp to 5 V o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"
- note removed: "J15 SERVO 24V and J17 SERVO UART: same pinout as CN5 / CN13 on the MES2 Harvester, so its cables fit. The FE-URT-2 turns the UART into the Feetech half-duplex servo bus and passes the 24 V on to the servos. UART on module USART2: PA2 TX → pin 4, pin 3 → PA3 RX (5 V-tolerant). Set the FE-URT-2 level switch to 3.3 V (not 5 V): it only sets the UART levels, the servo 24 V is unchanged. At 5 V its TX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"
- note removed: "U10 YLPTEC URB2405LD-20WR3: 9-36 V in, 5 V 4 A, 20 W isolated, short-circuit protected, 2" x 1" DIP. CTRL and Trim open (on, 5.0 V). C30 47 µF (datasheet C1 47-100 µF), C33 / C34 22 µF (C2 / C3 10-22 µF). F11 3 A PTC (same part as the relay outputs) + D22 SMF6.0A, then J16: the MES4-Flasher's USB-C power-only receptacle, rated 5 V 3 A (3 A on VBUS; GND pins 1.25 A each). R40 / R39 10k Rp to 5 V o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"
- moved on the sheet: R37
