File: MES4_Carrier_EC/Sensors.kicad_sch (KiCad schematic)
At the start: 14 parts, among them J10 SENS1, J11 SENS2, U7 PC817, U8 PC817

Commit message: Put relay coil feedback back on PA0-PA3 (MES4 GPIO standard)
All 14 module GPIOs now follow the MES4-CIF §2c table. The TCA9535 is
removed from the Relays 3-4 sheet and J1 fingers 43/45/47/49 drive the
relay 1-4 feedback dividers again. The winch relays are left undriven
(gate inputs no-connected, 100k pull-downs hold them off) until they
move to the TCA9535 + photoMOS design (HANDOFF.md step 2).

Removing U4 renumbers U5-U12 to U4-U11 and C15-C45 to C14-C44; the
README refs follow. Adds generator/checks.py (pin/pad, single-pin nets,
duplicate UUIDs, LCSC numbers), run by run.sh after ERC.

Co-Authored-By: Claude Opus 5.5 <noreply@anthropic.com>
Parts:
- removed C20: 100nF 50V, Capacitor_SMD:C_0603_1608Metric, symbol Device:C
- removed U8: PC817, Package_DIP:SMDIP-4_W9.53mm, symbol Isolator:PC817
- added C18: 100nF 50V, Capacitor_SMD:C_0603_1608Metric, symbol Device:C
- added U6: PC817, Package_DIP:SMDIP-4_W9.53mm, symbol Isolator:PC817
Connections:
- net +3V3_MOD: now also U6.4
- net GND_24V: now also C18.2, U6.2
- net PB6: now also U6.3; no longer U7.3
- net PC15: now also U7.3
- net SENS1_PWR: now also C18.1; no longer C19.1
- net SENS2_PWR: now also C19.1
- net at D18.1 (K), R32.2: now also U6.1; no longer U7.1
- net at D19.1 (K), R34.2: now also U7.1
Other:
- note added: "For 3-wire PNP (sourcing) 24 V sensors, e.g. Autonics PRD08 / PR series (brown +V, black OUT, blue 0 V). NPN (sinking) sensors need a different input circuit. Same circuit as the MES4-Flasher sensor channels 3 / 4 (PB6 / PC15), without the INA226 supply monitors. GPIO budget: all 14 module pins are used (Main sheet, MES4-CIF §2c). More sensors need inputs on I²C1, e.g. a TCA9535 expander (0x20-0x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"
- note added: "J10: 1 = +24 V (brown) through F7 100 mA PTC, 2 = sensor output (black), 3 = 0 V (blue). Output ON (24 V): ≈ 2.3 mA through R32 10k + U6 LED → PB6 HIGH (3.3 V, emitter follower). Output OFF, cable unplugged or broken: PB6 LOW (R33 10k pull-down). D18 1N4148W: reverse clamp across the opto LED. C18 100 nF / 50 V: supply decoupling + ESD. A shorted sensor cable trips F7 only: the other sensor and t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"
- note added: "J11: 1 = +24 V (brown) through F8 100 mA PTC, 2 = sensor output (black), 3 = 0 V (blue). Output ON (24 V): ≈ 2.3 mA through R34 10k + U7 LED → PC15 HIGH (3.3 V, emitter follower). Output OFF, cable unplugged or broken: PC15 LOW (R35 10k pull-down). D19 1N4148W: reverse clamp across the opto LED. C19 100 nF / 50 V: supply decoupling + ESD. A shorted sensor cable trips F8 only: the other sensor and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"
- note removed: "For 3-wire PNP (sourcing) 24 V sensors, e.g. Autonics PRD08 / PR series (brown +V, black OUT, blue 0 V). NPN (sinking) sensors need a different input circuit. Same circuit as the MES4-Flasher sensor channels 3 / 4 (PB6 / PC15), without the INA226 supply monitors. GPIO budget: all 14 module pins are used (Main sheet). More sensors can use the TCA9535 expander (Relays 3-4 sheet), which has 12 spare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"
- note removed: "J10: 1 = +24 V (brown) through F7 100 mA PTC, 2 = sensor output (black), 3 = 0 V (blue). Output ON (24 V): ≈ 2.3 mA through R32 10k + U7 LED → PB6 HIGH (3.3 V, emitter follower). Output OFF, cable unplugged or broken: PB6 LOW (R33 10k pull-down). D18 1N4148W: reverse clamp across the opto LED. C19 100 nF / 50 V: supply decoupling + ESD. A shorted sensor cable trips F7 only: the other sensor and t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"
- note removed: "J11: 1 = +24 V (brown) through F8 100 mA PTC, 2 = sensor output (black), 3 = 0 V (blue). Output ON (24 V): ≈ 2.3 mA through R34 10k + U8 LED → PC15 HIGH (3.3 V, emitter follower). Output OFF, cable unplugged or broken: PC15 LOW (R35 10k pull-down). D19 1N4148W: reverse clamp across the opto LED. C20 100 nF / 50 V: supply decoupling + ESD. A shorted sensor cable trips F8 only: the other sensor and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"

Commit message: Drop relay coil feedback; winch on PA0/PA1, servo on USART2
User decision: free the four feedback pins instead of adding an I²C
expander. The Flasher template's 10k/15k/10 nF dividers are removed from
all relay channels and relay diagnosis is INA226-only. PA0/PA1 drive the
IM03GR winch relays again and PA2/PA3 carry the door servo UART
(USART2), so the SC16IS740 bridge, its crystal and caps, and the unused
TCA9535 code are removed. This deliberately differs from the MES4-CIF
§2c GPIO table; the GPIO map, root notes, README and HANDOFF say so.

189 parts, ERC clean, checks.py passes. README refs follow the
renumbering.

Co-Authored-By: Claude Opus 5.5 <noreply@anthropic.com>
Parts:
- removed C18, C19: 100nF 50V, Capacitor_SMD:C_0603_1608Metric, symbol Device:C
- removed R32, R34: 10k, Resistor_SMD:R_0603_1608Metric, symbol Device:R
- removed R33, R35: 10k, Resistor_SMD:R_0402_1005Metric, symbol Device:R
- added C14, C15: 100nF 50V, Capacitor_SMD:C_0603_1608Metric, symbol Device:C
- added R24, R26: 10k, Resistor_SMD:R_0603_1608Metric, symbol Device:R
- added R25, R27: 10k, Resistor_SMD:R_0402_1005Metric, symbol Device:R
Connections:
- net GND: now also R25.2, R27.2
- net GND_24V: now also C14.2, C15.2
- net PB6: now also R25.1
- net PC15: now also R27.1
- net SENS1: now also R24.1
- net SENS1_PWR: now also C14.1
- net SENS2: now also R26.1
- net SENS2_PWR: now also C15.1
- net at D18.1 (K), U6.1: now also R24.2
- net at D19.1 (K), U7.1: now also R26.2
Other:
- note added: "J10: 1 = +24 V (brown) through F7 100 mA PTC, 2 = sensor output (black), 3 = 0 V (blue). Output ON (24 V): ≈ 2.3 mA through R24 10k + U6 LED → PB6 HIGH (3.3 V, emitter follower). Output OFF, cable unplugged or broken: PB6 LOW (R25 10k pull-down). D18 1N4148W: reverse clamp across the opto LED. C14 100 nF / 50 V: supply decoupling + ESD. A shorted sensor cable trips F7 only: the other sensor and t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"
- note added: "J11: 1 = +24 V (brown) through F8 100 mA PTC, 2 = sensor output (black), 3 = 0 V (blue). Output ON (24 V): ≈ 2.3 mA through R26 10k + U7 LED → PC15 HIGH (3.3 V, emitter follower). Output OFF, cable unplugged or broken: PC15 LOW (R27 10k pull-down). D19 1N4148W: reverse clamp across the opto LED. C15 100 nF / 50 V: supply decoupling + ESD. A shorted sensor cable trips F8 only: the other sensor and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"
- note removed: "J10: 1 = +24 V (brown) through F7 100 mA PTC, 2 = sensor output (black), 3 = 0 V (blue). Output ON (24 V): ≈ 2.3 mA through R32 10k + U6 LED → PB6 HIGH (3.3 V, emitter follower). Output OFF, cable unplugged or broken: PB6 LOW (R33 10k pull-down). D18 1N4148W: reverse clamp across the opto LED. C18 100 nF / 50 V: supply decoupling + ESD. A shorted sensor cable trips F7 only: the other sensor and t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"
- note removed: "J11: 1 = +24 V (brown) through F8 100 mA PTC, 2 = sensor output (black), 3 = 0 V (blue). Output ON (24 V): ≈ 2.3 mA through R34 10k + U7 LED → PC15 HIGH (3.3 V, emitter follower). Output OFF, cable unplugged or broken: PC15 LOW (R35 10k pull-down). D19 1N4148W: reverse clamp across the opto LED. C19 100 nF / 50 V: supply decoupling + ESD. A shorted sensor cable trips F8 only: the other sensor and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"

Commit message: Address design review R1: INA236, J15 polarity, review fixes
M1: U2-U5 are now TI INA236AIDDFR (C5443912, 50 V abs max, TSOT-23-8)
instead of the INA226 (40 V), since the SMBJ30A clamps at up to 48.4 V.
A project INA236 symbol keeps the INA226 body so the Flasher relay
wiring lands on the same pins; A1 and VBUS are gone (bus read on IN-),
addresses 0x40-0x43 via A0 = GND / VS / SDA / SCL. Same CONFIG / CAL /
MASK / ALERT values; notes give the 1.6 mV bus LSB and Device ID.
M3: J15 servo 24 V is pin 1 = +24 V like every power terminal.
L4: R38 servo RX series resistor 1k (limits PA3 back-feed).
L2: "current present" threshold 3 mA. L6: Power notes use 13 A / 2.2 W.
M2 / L5: silkscreen notes for "5V LOAD CELL - NEVER 24V" and
"CAN - NOT ETHERNET" (no keyed connector, by choice).
RJ45 1x4 footprint rebuilt from the HCTL drawing (14.0 mm ports,
Ø1.5 shield and Ø3.2 peg positions); U1 / U9 / U10 checked against the
JLC library and YLPTEC drawing. HANDOFF gains the review status table
and a layout checklist.

Co-Authored-By: Claude Opus 5.5 <noreply@anthropic.com>
Other:
- note added: "For 3-wire PNP (sourcing) 24 V sensors, e.g. Autonics PRD08 / PR series (brown +V, black OUT, blue 0 V). NPN (sinking) sensors need a different input circuit. Same circuit as the MES4-Flasher sensor channels 3 / 4 (PB6 / PC15), without the Flasher INA226 supply monitors. GPIO budget: all 14 module pins are used (Main sheet, MES4-CIF §2c). More sensors need inputs on I²C1, e.g. a TCA9535 expander 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"
- note removed: "For 3-wire PNP (sourcing) 24 V sensors, e.g. Autonics PRD08 / PR series (brown +V, black OUT, blue 0 V). NPN (sinking) sensors need a different input circuit. Same circuit as the MES4-Flasher sensor channels 3 / 4 (PB6 / PC15), without the INA226 supply monitors. GPIO budget: all 14 module pins are used (Main sheet, MES4-CIF §2c). More sensors need inputs on I²C1, e.g. a TCA9535 expander (0x20-0x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"

Commit message: One ground and a 4-layer board
- GND_24V merged into GND (ONE_GND in gen.py): every GND_24V power symbol
  becomes GND, net tie NT1 left out, notes reworded. Symbol UUIDs unchanged,
  so every footprint keeps its link.
- 4 layers, JLC04161H-7628 stackup (1.6 mm, ENIG): Top Signal / GND plane
  (In1) / +24V plane (In2) / Bottom Signal.
- Net classes: Out_3A (1.5 mm) for +24V_SRV, +5V_SCR, VBUS_SCR; +24V_AUX to
  24V_Power; +5V_SRV, +9V_IMU, IMU_9V to Power; INA236 shunt pattern fixed
  (Net-(U*-IN-)).
- J1's NPTH holes back to F&B.Cu as in its library footprint.

ERC 0, checks passed, DRC 11 silkscreen warnings, schematic parity clean.

Co-Authored-By: Claude Opus 5.5 <noreply@anthropic.com>
Connections:
- net GND_24V is gone; now on net GND: C14.2, C15.2, D18.2 (A), D19.2 (A), J10.3 (Pin_3), J11.3 (Pin_3), U6.2, U7.2
