File: MES4_Carrier_EC/Winch.kicad_sch (KiCad schematic)
At the start: 17 parts, among them J18 WINCH, K5 IM03GR, K6 IM03GR, Q6 AO3400A, Q7 AO3400A, U12 SC16IS740IPW, Y1 16MHz

Commit message: Put relay coil feedback back on PA0-PA3 (MES4 GPIO standard)
All 14 module GPIOs now follow the MES4-CIF §2c table. The TCA9535 is
removed from the Relays 3-4 sheet and J1 fingers 43/45/47/49 drive the
relay 1-4 feedback dividers again. The winch relays are left undriven
(gate inputs no-connected, 100k pull-downs hold them off) until they
move to the TCA9535 + photoMOS design (HANDOFF.md step 2).

Removing U4 renumbers U5-U12 to U4-U11 and C15-C45 to C14-C44; the
README refs follow. Adds generator/checks.py (pin/pad, single-pin nets,
duplicate UUIDs, LCSC numbers), run by run.sh after ERC.

Co-Authored-By: Claude Opus 5.5 <noreply@anthropic.com>
Parts:
- removed C43: 100nF, Capacitor_SMD:C_0402_1005Metric, symbol Device:C
- removed C45: 12pF, Capacitor_SMD:C_0402_1005Metric, symbol Device:C
- removed K6: IM03GR, MES4-Carrier-EC:RELAY-SMD_IMXXGR, symbol MES4-Carrier-EC:IM03GR
- removed Q6: AO3400A, Package_TO_SOT_SMD:SOT-23, symbol Transistor_FET:AO3400A
- removed U12: SC16IS740IPW, Package_SO:TSSOP-16_4.4x5mm_P0.65mm, symbol Interface_UART:SC16IS740
- added C42: 100nF, Capacitor_SMD:C_0402_1005Metric, symbol Device:C
- added D25: 1N4148W, Diode_SMD:D_SOD-123, symbol Device:D
- added R51: 100k, Resistor_SMD:R_0402_1005Metric, symbol Device:R
- added U11: SC16IS740IPW, Package_SO:TSSOP-16_4.4x5mm_P0.65mm, symbol Interface_UART:SC16IS740
- added Y1: 16MHz, Crystal:Crystal_SMD_3225-4Pin_3.2x2.5mm, symbol Device:Crystal_GND24
- C43: renamed from Y1; value 16MHz -> 12pF; footprint Crystal:Crystal_SMD_3225-4Pin_3.2x2.5mm -> Capacitor_SMD:C_0402_1005Metric; symbol Device:Crystal_GND24 -> Device:C; LCSC C13738 -> C1547
- K6: renamed from R51; value 100k -> IM03GR; footprint Resistor_SMD:R_0402_1005Metric -> MES4-Carrier-EC:RELAY-SMD_IMXXGR; symbol Device:R -> MES4-Carrier-EC:IM03GR; LCSC C25741 -> C2153100
- Q6: renamed from D25; value 1N4148W -> AO3400A; footprint Diode_SMD:D_SOD-123 -> Package_TO_SOT_SMD:SOT-23; symbol Device:D -> Transistor_FET:AO3400A; LCSC C81598 -> C20917
Connections:
- net +3V3_MOD: now also C42.1, U11.1 (VDD), U11.2 (A0/~{CS}), U11.3 (A1/SI), U11.8 (I2C/~{SPI})
- net +5V_24: now also K6.1 (COIL+), D25.1 (K); no longer Q6.1 (K)
- net GND: now also Q6.2 (S), C42.2, R51.2, U11.11 (~{CTS}), U11.9 (VSS), Y1.2, Y1.4; no longer C43.4, K6.2
- net I2C1_SCL: now also U11.5 (SCL/SCLK)
- net I2C1_SDA: now also U11.6 (SDA)
- net ILK_ACLK: now also K6.3 (COM1)
- net ILK_CLK: now also K6.7 (NC2)
- net SRV_UART_RX: now also U11.13 (RX)
- net SRV_UART_TX: now also U11.12 (TX)
- net WINCH_ACLK: now also K6.4 (NO1)
- net WINCH_COM: now also K6.6 (COM2)
- net at R54.2: now also U11.14 (~{RESET})
- net at C43.1: now also U11.15 (XTAL1), Y1.1; no longer C44.1
- net at K5.8 (COIL-): now also Q6.3 (D), D25.2 (A); no longer Q6.2 (A)
- net at D26.2 (A), Q7.3 (D): now also K6.8 (COIL-)
- net at R50.2: now also Q6.1 (G), R51.1; no longer K6.1
- net PA0: no longer names the net of R50.1
- net PA1: no longer names the net of R52.1
- new net: C44.1, U11.16 (XTAL2), Y1.3
- no-connect marks 7 -> 9
Other:
- note added: "U11 NXP SC16IS740IPW: I²C1 slave at 0x48 (A1 = A0 = VDD; INA226s 0x40-0x45, TCA9535 0x20). TX / RX → servo UART terminal (AuxPower sheet, 100 Ω + ESD there) → FE-URT-2. Y1 16 MHz (CL 9 pF) + C43 / C44 12 pF: baud = 16 MHz / (16 × divisor): 1 Mbit/s (Feetech default, divisor 1), 500k (2), 250k (4) are exact. IRQ not connected (no module pin free): poll the LSR / RXLVL registers. CTS tied low (alwa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"
- note removed: "U12 NXP SC16IS740IPW: I²C1 slave at 0x48 (A1 = A0 = VDD; INA226s 0x40-0x45, TCA9535 0x20). TX / RX → servo UART terminal (AuxPower sheet, 100 Ω + ESD there) → FE-URT-2. Y1 16 MHz (CL 9 pF) + C44 / C45 12 pF: baud = 16 MHz / (16 × divisor): 1 Mbit/s (Feetech default, divisor 1), 500k (2), 250k (4) are exact. IRQ not connected (no module pin free): poll the LSR / RXLVL registers. CTS tied low (alwa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"

Commit message: Drop relay coil feedback; winch on PA0/PA1, servo on USART2
User decision: free the four feedback pins instead of adding an I²C
expander. The Flasher template's 10k/15k/10 nF dividers are removed from
all relay channels and relay diagnosis is INA226-only. PA0/PA1 drive the
IM03GR winch relays again and PA2/PA3 carry the door servo UART
(USART2), so the SC16IS740 bridge, its crystal and caps, and the unused
TCA9535 code are removed. This deliberately differs from the MES4-CIF
§2c GPIO table; the GPIO map, root notes, README and HANDOFF say so.

189 parts, ERC clean, checks.py passes. README refs follow the
renumbering.

Co-Authored-By: Claude Opus 5.5 <noreply@anthropic.com>
Parts:
- removed C42: 100nF, Capacitor_SMD:C_0402_1005Metric, symbol Device:C
- removed C43, C44: 12pF, Capacitor_SMD:C_0402_1005Metric, symbol Device:C
- removed R50, R52: 100Ω, Resistor_SMD:R_0402_1005Metric, symbol Device:R
- removed R51, R53: 100k, Resistor_SMD:R_0402_1005Metric, symbol Device:R
- removed R54: 10k, Resistor_SMD:R_0402_1005Metric, symbol Device:R
- removed U11: SC16IS740IPW, Package_SO:TSSOP-16_4.4x5mm_P0.65mm, symbol Interface_UART:SC16IS740
- removed Y1: 16MHz, Crystal:Crystal_SMD_3225-4Pin_3.2x2.5mm, symbol Device:Crystal_GND24
- added R42, R44: 100Ω, Resistor_SMD:R_0402_1005Metric, symbol Device:R
- added R43, R45: 100k, Resistor_SMD:R_0402_1005Metric, symbol Device:R
Connections:
- net GND: now also R43.2, R45.2
- net at Q6.1 (G): now also R42.2, R43.1
- net at Q7.1 (G): now also R44.2, R45.1
- new net PA0: R42.1
- new net PA1: R44.1
- no-connect marks 9 -> 4
Other:
- note removed: "Servo UART: SC16IS740 I²C-UART bridge (I²C1 0x48)"
- note removed: "U11 NXP SC16IS740IPW: I²C1 slave at 0x48 (A1 = A0 = VDD; INA226s 0x40-0x45, TCA9535 0x20). TX / RX → servo UART terminal (AuxPower sheet, 100 Ω + ESD there) → FE-URT-2. Y1 16 MHz (CL 9 pF) + C43 / C44 12 pF: baud = 16 MHz / (16 × divisor): 1 Mbit/s (Feetech default, divisor 1), 500k (2), 250k (4) are exact. IRQ not connected (no module pin free): poll the LSR / RXLVL registers. CTS tied low (alwa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"

Commit message: Isolate the 48 V winch side, add servo TX pull-up, tidy block diagram
Winch: J18 and the WINCH_* / ILK_* nets already touch only relay
contacts; they now form net class Winch_48V (0.6 mm clearance), and the
Winch sheet, README and HANDOFF state the isolation rules (>= 2 mm to
other copper, no GND pour under J18, no ESD to GND on J18).

Servo: R37 10k pull-up holds PA2 (TX) idle HIGH while the MCU is in
reset. AuxPower/Winch refs R37-R45 shift by one; README follows, and the
LED8 resistor ref is corrected to R35.

Block diagram: door servo block, winch and servo links from the module,
24 V routed so it never crosses a signal line, channel lines on an even
5.08 mm pitch.

Co-Authored-By: Claude Opus 5.5 <noreply@anthropic.com>
Parts:
- removed R42: 100Ω, Resistor_SMD:R_0402_1005Metric, symbol Device:R
- added R46: 100k, Resistor_SMD:R_0402_1005Metric, symbol Device:R
- R43, R45: value 100k -> 100Ω; LCSC C25741 -> C25076
- R44: value 100Ω -> 100k; LCSC C25076 -> C25741
Connections:
- net GND: now also R44.2, R46.2; no longer R43.2, R45.2
- net PA0: now also R43.1
- net PA1: now also R45.1; no longer R44.1
- net at Q6.1 (G): now also R43.2, R44.1; no longer R43.1
- new net: Q7.1 (G), R45.2, R46.1
Changed lines of the file:
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@@
 		(effects (font (size 2 2) (bold yes)) (justify left top))
 	)
-	(text "Same relays and terminal as the MES2_Extension \"WINCH CONTROL\": TE IM03GR, 5 V coil (178 Ω, 28 mA) from\n+5V_24, contacts 2 A / 220 VDC, 60 W DC. They only switch the 48 V winch controller's direction inputs to\nJ18 pin 2 (COM): pin 1 = CLK, pin 3 = ACLK. They are not rated for the winch motor current.\nTE terminal assignment: coil 1 (+) / 8 (-); pole 1: 3 COM, 2 NC, 4 NO; pole 2: 6 COM, 7 NC, 5 NO.\n\nDrivers as on the relay sheets (CIF §7a): AO3400A, 100 Ω gate, 100k pull-down, so both relays are OFF\nduring reset and boot (PA0 / PA1 float then). The Extension used 2SC2884 transistors without a pull-down.\n\nHardware interlock (new, uses the spare second pole): CLK closes COM → ILK_CLK → K5 NO1 → CLK only\nwhile K6 rests (its NC2 feeds ILK_CLK), and the same the other way. If both relays are energised, both\noutputs stay open, so the winch can never see both directions at once. Firmware still drives only one.\n\nPA0 / PA1 are relay 1 / 2 coil feedback in the MES4-CIF §2c table. This board drops the coil feedback\nto free them for the winch (E-Crawler GPIO budget)."
+	(text "Same relays and terminal as the MES2_Extension \"WINCH CONTROL\": TE IM03GR, 5 V coil (178 Ω, 28 mA) from\n+5V_24, contacts 2 A / 220 VDC, 60 W DC. They only switch the 48 V winch controller's direction inputs to\nJ18 pin 2 (COM): pin 1 = CLK, pin 3 = ACLK. They are not rated for the winch motor current.\nTE terminal assignment: coil 1 (+) / 8 (-); pole 1: 3 COM, 2 NC, 4 NO; pole 2: 6 COM, 7 NC, 5 NO.\n\nDrivers as on the relay sheets (CIF §7a): AO3400A, 100 Ω gate, 100k pull-down, so both relays are OFF\nduring reset and boot (PA0 / PA1 float then). The Extension used 2SC2884 transistors without a pull-down.\n\nHardware interlock (new, uses the spare second pole): CLK closes COM → ILK_CLK → K5 NO1 → CLK only\nwhile K6 rests (its NC2 feeds ILK_CLK), and the same the other way. If both relays are energised, both\noutputs stay open, so the winch can never see both directions at once. Firmware still drives only one.\n\nIsolation from the 48 V winch system: J18 and the WINCH_ / ILK_ nets touch only relay contacts. No carrier\nGND, supply or ESD clamp connects to that side, so the relays' coil-to-contact insulation is the barrier\n(TE IM series, up to 2500 Vrms). PCB: net class Winch_48V; keep ≥ 2 mm from all other copper and no GND\npour under J18 or the contact pins. Never add a TVS / ESD diode to GND on J18: it bridges the isolation.\n\nPA0 / PA1 are relay 1 / 2 coil feedback in the MES4-CIF §2c table. This board drops the coil feedback\nto free them for the winch (E-Crawler GPIO budget)."
 		(exclude_from_sim no)
 		(at 17.78 156.21 0)
@@
 		(instances
 			(project "MES4_Carrier_EC"
-				(path "/da774ca2-fff6-5e5d-8e21-ede9d04ec2cb/0959b9ec-5a3a-5f07-b996-83d523c173ff"
+				(path "/0370b922-a365-5c71-ab6f-f5cfbc7b5e5a/1faebd9f-5ef7-5632-999b-932f8eeca23c"
 					(reference "K5")
 					(unit 1)
@@
 		(on_board yes)
 		(dnp no)
-		(property "Reference" "#PWR168"
+		(property "Reference" "#PWR169"
 			(at 83.82 50.8 0)
 			(effects (font (size 1.27 1.27)) (hide yes))
@@
 		(instances
 			(project "MES4_Carrier_EC"
-				(path "/da774ca2-fff6-5e5d-8e21-ede9d04ec2cb/0959b9ec-5a3a-5f07-b996-83d523c173ff"
-					(reference "#PWR168")
+				(path "/0370b922-a365-5c71-ab6f-f5cfbc7b5e5a/1faebd9f-5ef7-5632-999b-932f8eeca23c"
+					(reference "#PWR169")
 					(unit 1)
 				)
@@
 		(instances
 			(project "MES4_Carrier_EC"
-				(path "/da774ca2-fff6-5e5d-8e21-ede9d04ec2cb/0959b9ec-5a3a-5f07-b996-83d523c173ff"
+				(path "/0370b922-a365-5c71-ab6f-f5cfbc7b5e5a/1faebd9f-5ef7-5632-999b-932f8eeca23c"
 					(reference "D25")
 					(unit 1)
@@
 		(instances
 			(project "MES4_Carrier_EC"
-				(path "/da774ca2-fff6-5e5d-8e21-ede9d04ec2cb/0959b9ec-5a3a-5f07-b996-83d523c173ff"
+				(path "/0370b922-a365-5c71-ab6f-f5cfbc7b5e5a/1faebd9f-5ef7-5632-999b-932f8eeca23c"
 					(reference "Q6")
 					(unit 1)
@@
 		(on_board yes)
 		(dnp no)
-		(property "Reference" "#PWR169"
+		(property "Reference" "#PWR170"
 			(at 88.9 78.74 0)
 			(effects (font (size 1.27 1.27)) (hide yes))
@@
 		(instances
 			(project "MES4_Carrier_EC"
-				(path "/da774ca2-fff6-5e5d-8e21-ede9d04ec2cb/0959b9ec-5a3a-5f07-b996-83d523c173ff"
-					(reference "#PWR169")
+				(path "/0370b922-a365-5c71-ab6f-f5cfbc7b5e5a/1faebd9f-5ef7-5632-999b-932f8eeca23c"
+					(reference "#PWR170")
 					(unit 1)
 				)
@@
 		(on_board yes)
 		(dnp no)
-		(property "Reference" "R42"
+		(property "Reference" "R43"
 			(at 67.31 69.85 90)
 			(effects (font (size 1.27 1.27)))
@@
 		(instances
 			(project "MES4_Carrier_EC"
-				(path "/da774ca2-fff6-5e5d-8e21-ede9d04ec2cb/0959b9ec-5a3a-5f07-b996-83d523c173ff"
-					(reference "R42")
+				(path "/0370b922-a365-5c71-ab6f-f5cfbc7b5e5a/1faebd9f-5ef7-5632-999b-932f8eeca23c"
+					(reference "R43")
 					(unit 1)
 				)
@@
 		(on_board yes)
 		(dnp no)
-		(property "Reference" "R43"
+		(property "Reference" "R44"
 			(at 76.2 76.2 0)
 			(effects (font (size 1.27 1.27)) (justify right))
@@
 		(instances
 			(project "MES4_Carrier_EC"
-				(path "/da774ca2-fff6-5e5d-8e21-ede9d04ec2cb/0959b9ec-5a3a-5f07-b996-83d523c173ff"
-					(reference "R43")
+				(path "/0370b922-a365-5c71-ab6f-f5cfbc7b5e5a/1faebd9f-5ef7-5632-999b-932f8eeca23c"
+					(reference "R44")
 					(unit 1)
 				)
@@
 		(on_board yes)
 		(dnp no)
-		(property "Reference" "#PWR170"
+		(property "Reference" "#PWR171"
 			(at 78.74 81.28 0)
 			(effects (font (size 1.27 1.27)) (hide yes))
@@
 		(instances
 			(project "MES4_Carrier_EC"
-				(path "/da774ca2-fff6-5e5d-8e21-ede9d04ec2cb/0959b9ec-5a3a-5f07-b996-83d523c173ff"
-					(reference "#PWR170")
+				(path "/0370b922-a365-5c71-ab6f-f5cfbc7b5e5a/1faebd9f-5ef7-5632-999b-932f8eeca23c"
+					(reference "#PWR171")
 					(unit 1)
 				)
@@
 		(instances
 			(project "MES4_Carrier_EC"
-				(path "/da774ca2-fff6-5e5d-8e21-ede9d04ec2cb/0959b9ec-5a3a-5f07-b996-83d523c173ff"
+				(path "/0370b922-a365-5c71-ab6f-f5cfbc7b5e5a/1faebd9f-5ef7-5632-999b-932f8eeca23c"
 					(reference "K6")
 					(unit 1)
@@
 		(on_board yes)
 		(dnp no)
-		(property "Reference" "#PWR171"
+		(property "Reference" "#PWR172"
 			(at 83.82 101.6 0)
 			(effects (font (size 1.27 1.27)) (hide yes))
@@
 		(instances
 			(project "MES4_Carrier_EC"
-				(path "/da774ca2-fff6-5e5d-8e21-ede9d04ec2cb/0959b9ec-5a3a-5f07-b996-83d523c173ff"
-					(reference "#PWR171")
+				(path "/0370b922-a365-5c71-ab6f-f5cfbc7b5e5a/1faebd9f-5ef7-5632-999b-932f8eeca23c"
+					(reference "#PWR172")
 					(unit 1)
 				)
@@
 		(instances
 			(project "MES4_Carrier_EC"
-				(path "/da774ca2-fff6-5e5d-8e21-ede9d04ec2cb/0959b9ec-5a3a-5f07-b996-83d523c173ff"
+				(path "/0370b922-a365-5c71-ab6f-f5cfbc7b5e5a/1faebd9f-5ef7-5632-999b-932f8eeca23c"
 					(reference "D26")
 					(unit 1)
@@
 		(instances
 			(project "MES4_Carrier_EC"
-				(path "/da774ca2-fff6-5e5d-8e21-ede9d04ec2cb/0959b9ec-5a3a-5f07-b996-83d523c173ff"
+				(path "/0370b922-a365-5c71-ab6f-f5cfbc7b5e5a/1faebd9f-5ef7-5632-999b-932f8eeca23c"
 					(reference "Q7")
 					(unit 1)
@@
 		(on_board yes)
 		(dnp no)
-		(property "Reference" "#PWR172"
+		(property "Reference" "#PWR173"
 			(at 88.9 129.54 0)
 			(effects (font (size 1.27 1.27)) (hide yes))
@@
 		(instances
 			(project "MES4_Carrier_EC"
-				(path "/da774ca2-fff6-5e5d-8e21-ede9d04ec2cb/0959b9ec-5a3a-5f07-b996-83d523c173ff"
-					(reference "#PWR172")
+				(path "/0370b922-a365-5c71-ab6f-f5cfbc7b5e5a/1faebd9f-5ef7-5632-999b-932f8eeca23c"
+					(reference "#PWR173")
 					(unit 1)
 				)
@@
 		(on_board yes)
 		(dnp no)
-		(property "Reference" "R44"
+		(property "Reference" "R45"
 			(at 67.31 120.65 90)
 			(effects (font (size 1.27 1.27)))
@@
 		(instances
 			(project "MES4_Carrier_EC"
-				(path "/da774ca2-fff6-5e5d-8e21-ede9d04ec2cb/0959b9ec-5a3a-5f07-b996-83d523c173ff"
-					(reference "R44")
+				(path "/0370b922-a365-5c71-ab6f-f5cfbc7b5e5a/1faebd9f-5ef7-5632-999b-932f8eeca23c"
+					(reference "R45")
 					(unit 1)
 				)
@@
 		(on_board yes)
 		(dnp no)
-		(property "Reference" "R45"
+		(property "Reference" "R46"
 			(at 76.2 127 0)
 			(effects (font (size 1.27 1.27)) (justify right))
@@
 		(instances
 			(project "MES4_Carrier_EC"
-				(path "/da774ca2-fff6-5e5d-8e21-ede9d04ec2cb/0959b9ec-5a3a-5f07-b996-83d523c173ff"
-					(reference "R45")
+				(path "/0370b922-a365-5c71-ab6f-f5cfbc7b5e5a/1faebd9f-5ef7-5632-999b-932f8eeca23c"
+					(reference "R46")
 					(unit 1)
 				)
@@
 		(on_board yes)
 		(dnp no)
-		(property "Reference" "#PWR173"
+		(property "Reference" "#PWR174"
 			(at 78.74 132.08 0)
 			(effects (font (size 1.27 1.27)) (hide yes))
@@
 		(instances
 			(project "MES4_Carrier_EC"
-				(path "/da774ca2-fff6-5e5d-8e21-ede9d04ec2cb/0959b9ec-5a3a-5f07-b996-83d523c173ff"
-					(reference "#PWR173")
+				(path "/0370b922-a365-5c71-ab6f-f5cfbc7b5e5a/1faebd9f-5ef7-5632-999b-932f8eeca23c"
+					(reference "#PWR174")
 					(unit 1)
 				)
@@
 		(instances
 			(project "MES4_Carrier_EC"
-				(path "/da774ca2-fff6-5e5d-8e21-ede9d04ec2cb/0959b9ec-5a3a-5f07-b996-83d523c173ff"
+				(path "/0370b922-a365-5c71-ab6f-f5cfbc7b5e5a/1faebd9f-5ef7-5632-999b-932f8eeca23c"
 					(reference "J18")
 					(unit 1)
