File: MES4_Carrier_EC/Winch.kicad_sch (KiCad schematic)
At the start: 11 parts, among them J18 WINCH, K5 IM03GR, K6 IM03GR, Q6 AO3400A, Q7 AO3400A

Commit message: Address design review R1: INA236, J15 polarity, review fixes
M1: U2-U5 are now TI INA236AIDDFR (C5443912, 50 V abs max, TSOT-23-8)
instead of the INA226 (40 V), since the SMBJ30A clamps at up to 48.4 V.
A project INA236 symbol keeps the INA226 body so the Flasher relay
wiring lands on the same pins; A1 and VBUS are gone (bus read on IN-),
addresses 0x40-0x43 via A0 = GND / VS / SDA / SCL. Same CONFIG / CAL /
MASK / ALERT values; notes give the 1.6 mV bus LSB and Device ID.
M3: J15 servo 24 V is pin 1 = +24 V like every power terminal.
L4: R38 servo RX series resistor 1k (limits PA3 back-feed).
L2: "current present" threshold 3 mA. L6: Power notes use 13 A / 2.2 W.
M2 / L5: silkscreen notes for "5V LOAD CELL - NEVER 24V" and
"CAN - NOT ETHERNET" (no keyed connector, by choice).
RJ45 1x4 footprint rebuilt from the HCTL drawing (14.0 mm ports,
Ø1.5 shield and Ø3.2 peg positions); U1 / U9 / U10 checked against the
JLC library and YLPTEC drawing. HANDOFF gains the review status table
and a layout checklist.

Co-Authored-By: Claude Opus 5.5 <noreply@anthropic.com>
Parts:
- removed K5, K6: IM03GR, MES4-Carrier-EC:RELAY-SMD_IMXXGR, symbol MES4-Carrier-EC:IM03GR
- added Q6, Q7: AO3400A, Package_TO_SOT_SMD:SOT-23, symbol Transistor_FET:AO3400A
- K5: renamed from Q6; value AO3400A -> IM03GR; footprint Package_TO_SOT_SMD:SOT-23 -> MES4-Carrier-EC:RELAY-SMD_IMXXGR; symbol Transistor_FET:AO3400A -> MES4-Carrier-EC:IM03GR; LCSC C20917 -> C2153100
- K6: renamed from Q7; value AO3400A -> IM03GR; footprint Package_TO_SOT_SMD:SOT-23 -> MES4-Carrier-EC:RELAY-SMD_IMXXGR; symbol Transistor_FET:AO3400A -> MES4-Carrier-EC:IM03GR; LCSC C20917 -> C2153100
Connections:
- net +5V_24: now also K5.1 (COIL+), K6.1 (COIL+)
- net GND: now also Q6.2 (S), Q7.2 (S); no longer K5.2 (S), K6.2 (S)
- net ILK_ACLK: now also K5.7 (NC2), K6.3 (COM1)
- net ILK_CLK: now also K5.3 (COM1), K6.7 (NC2)
- net WINCH_ACLK: now also K6.4 (NO1)
- net WINCH_CLK: now also K5.4 (NO1)
- net WINCH_COM: now also K5.6 (COM2), K6.6 (COM2)
- net at R45.2, R46.1: now also Q7.1 (G); no longer K6.1 (G)
- net at D26.2 (A): now also K6.8 (COIL-), Q7.3 (D); no longer K6.3 (D)
- net at R43.2, R44.1: now also Q6.1 (G); no longer K5.1 (G)
- net at D25.2 (A): now also K5.8 (COIL-), Q6.3 (D); no longer K5.3 (D)
Changed lines of the file:
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@@
 		(instances
 			(project "MES4_Carrier_EC"
-				(path "/0370b922-a365-5c71-ab6f-f5cfbc7b5e5a/1faebd9f-5ef7-5632-999b-932f8eeca23c"
+				(path "/0d8fbf0e-dd62-5be6-8889-307c6423adb0/ab87f4c8-555d-52c8-a423-b1818ccd4582"
 					(reference "K5")
 					(unit 1)
@@
 		(on_board yes)
 		(dnp no)
-		(property "Reference" "#PWR169"
+		(property "Reference" "#PWR163"
 			(at 83.82 50.8 0)
 			(effects (font (size 1.27 1.27)) (hide yes))
@@
 		(instances
 			(project "MES4_Carrier_EC"
-				(path "/0370b922-a365-5c71-ab6f-f5cfbc7b5e5a/1faebd9f-5ef7-5632-999b-932f8eeca23c"
-					(reference "#PWR169")
+				(path "/0d8fbf0e-dd62-5be6-8889-307c6423adb0/ab87f4c8-555d-52c8-a423-b1818ccd4582"
+					(reference "#PWR163")
 					(unit 1)
 				)
@@
 		(instances
 			(project "MES4_Carrier_EC"
-				(path "/0370b922-a365-5c71-ab6f-f5cfbc7b5e5a/1faebd9f-5ef7-5632-999b-932f8eeca23c"
+				(path "/0d8fbf0e-dd62-5be6-8889-307c6423adb0/ab87f4c8-555d-52c8-a423-b1818ccd4582"
 					(reference "D25")
 					(unit 1)
@@
 		(instances
 			(project "MES4_Carrier_EC"
-				(path "/0370b922-a365-5c71-ab6f-f5cfbc7b5e5a/1faebd9f-5ef7-5632-999b-932f8eeca23c"
+				(path "/0d8fbf0e-dd62-5be6-8889-307c6423adb0/ab87f4c8-555d-52c8-a423-b1818ccd4582"
 					(reference "Q6")
 					(unit 1)
@@
 		(on_board yes)
 		(dnp no)
-		(property "Reference" "#PWR170"
+		(property "Reference" "#PWR164"
 			(at 88.9 78.74 0)
 			(effects (font (size 1.27 1.27)) (hide yes))
@@
 		(instances
 			(project "MES4_Carrier_EC"
-				(path "/0370b922-a365-5c71-ab6f-f5cfbc7b5e5a/1faebd9f-5ef7-5632-999b-932f8eeca23c"
-					(reference "#PWR170")
+				(path "/0d8fbf0e-dd62-5be6-8889-307c6423adb0/ab87f4c8-555d-52c8-a423-b1818ccd4582"
+					(reference "#PWR164")
 					(unit 1)
 				)
@@
 		(instances
 			(project "MES4_Carrier_EC"
-				(path "/0370b922-a365-5c71-ab6f-f5cfbc7b5e5a/1faebd9f-5ef7-5632-999b-932f8eeca23c"
+				(path "/0d8fbf0e-dd62-5be6-8889-307c6423adb0/ab87f4c8-555d-52c8-a423-b1818ccd4582"
 					(reference "R43")
 					(unit 1)
@@
 		(instances
 			(project "MES4_Carrier_EC"
-				(path "/0370b922-a365-5c71-ab6f-f5cfbc7b5e5a/1faebd9f-5ef7-5632-999b-932f8eeca23c"
+				(path "/0d8fbf0e-dd62-5be6-8889-307c6423adb0/ab87f4c8-555d-52c8-a423-b1818ccd4582"
 					(reference "R44")
 					(unit 1)
@@
 		(on_board yes)
 		(dnp no)
-		(property "Reference" "#PWR171"
+		(property "Reference" "#PWR165"
 			(at 78.74 81.28 0)
 			(effects (font (size 1.27 1.27)) (hide yes))
@@
 		(instances
 			(project "MES4_Carrier_EC"
-				(path "/0370b922-a365-5c71-ab6f-f5cfbc7b5e5a/1faebd9f-5ef7-5632-999b-932f8eeca23c"
-					(reference "#PWR171")
+				(path "/0d8fbf0e-dd62-5be6-8889-307c6423adb0/ab87f4c8-555d-52c8-a423-b1818ccd4582"
+					(reference "#PWR165")
 					(unit 1)
 				)
@@
 		(instances
 			(project "MES4_Carrier_EC"
-				(path "/0370b922-a365-5c71-ab6f-f5cfbc7b5e5a/1faebd9f-5ef7-5632-999b-932f8eeca23c"
+				(path "/0d8fbf0e-dd62-5be6-8889-307c6423adb0/ab87f4c8-555d-52c8-a423-b1818ccd4582"
 					(reference "K6")
 					(unit 1)
@@
 		(on_board yes)
 		(dnp no)
-		(property "Reference" "#PWR172"
+		(property "Reference" "#PWR166"
 			(at 83.82 101.6 0)
 			(effects (font (size 1.27 1.27)) (hide yes))
@@
 		(instances
 			(project "MES4_Carrier_EC"
-				(path "/0370b922-a365-5c71-ab6f-f5cfbc7b5e5a/1faebd9f-5ef7-5632-999b-932f8eeca23c"
-					(reference "#PWR172")
+				(path "/0d8fbf0e-dd62-5be6-8889-307c6423adb0/ab87f4c8-555d-52c8-a423-b1818ccd4582"
+					(reference "#PWR166")
 					(unit 1)
 				)
@@
 		(instances
 			(project "MES4_Carrier_EC"
-				(path "/0370b922-a365-5c71-ab6f-f5cfbc7b5e5a/1faebd9f-5ef7-5632-999b-932f8eeca23c"
+				(path "/0d8fbf0e-dd62-5be6-8889-307c6423adb0/ab87f4c8-555d-52c8-a423-b1818ccd4582"
 					(reference "D26")
 					(unit 1)
@@
 		(instances
 			(project "MES4_Carrier_EC"
-				(path "/0370b922-a365-5c71-ab6f-f5cfbc7b5e5a/1faebd9f-5ef7-5632-999b-932f8eeca23c"
+				(path "/0d8fbf0e-dd62-5be6-8889-307c6423adb0/ab87f4c8-555d-52c8-a423-b1818ccd4582"
 					(reference "Q7")
 					(unit 1)
@@
 		(on_board yes)
 		(dnp no)
-		(property "Reference" "#PWR173"
+		(property "Reference" "#PWR167"
 			(at 88.9 129.54 0)
 			(effects (font (size 1.27 1.27)) (hide yes))
@@
 		(instances
 			(project "MES4_Carrier_EC"
-				(path "/0370b922-a365-5c71-ab6f-f5cfbc7b5e5a/1faebd9f-5ef7-5632-999b-932f8eeca23c"
-					(reference "#PWR173")
+				(path "/0d8fbf0e-dd62-5be6-8889-307c6423adb0/ab87f4c8-555d-52c8-a423-b1818ccd4582"
+					(reference "#PWR167")
 					(unit 1)
 				)
@@
 		(instances
 			(project "MES4_Carrier_EC"
-				(path "/0370b922-a365-5c71-ab6f-f5cfbc7b5e5a/1faebd9f-5ef7-5632-999b-932f8eeca23c"
+				(path "/0d8fbf0e-dd62-5be6-8889-307c6423adb0/ab87f4c8-555d-52c8-a423-b1818ccd4582"
 					(reference "R45")
 					(unit 1)
@@
 		(instances
 			(project "MES4_Carrier_EC"
-				(path "/0370b922-a365-5c71-ab6f-f5cfbc7b5e5a/1faebd9f-5ef7-5632-999b-932f8eeca23c"
+				(path "/0d8fbf0e-dd62-5be6-8889-307c6423adb0/ab87f4c8-555d-52c8-a423-b1818ccd4582"
 					(reference "R46")
 					(unit 1)
@@
 		(on_board yes)
 		(dnp no)
-		(property "Reference" "#PWR174"
+		(property "Reference" "#PWR168"
 			(at 78.74 132.08 0)
 			(effects (font (size 1.27 1.27)) (hide yes))
@@
 		(instances
 			(project "MES4_Carrier_EC"
-				(path "/0370b922-a365-5c71-ab6f-f5cfbc7b5e5a/1faebd9f-5ef7-5632-999b-932f8eeca23c"
-					(reference "#PWR174")
+				(path "/0d8fbf0e-dd62-5be6-8889-307c6423adb0/ab87f4c8-555d-52c8-a423-b1818ccd4582"
+					(reference "#PWR168")
 					(unit 1)
 				)
@@
 		(instances
 			(project "MES4_Carrier_EC"
-				(path "/0370b922-a365-5c71-ab6f-f5cfbc7b5e5a/1faebd9f-5ef7-5632-999b-932f8eeca23c"
+				(path "/0d8fbf0e-dd62-5be6-8889-307c6423adb0/ab87f4c8-555d-52c8-a423-b1818ccd4582"
 					(reference "J18")
 					(unit 1)
