File: MES4_Carrier_EC/Power.kicad_sch (KiCad schematic)
At the start: 29 parts, among them J5 24V IN, Q1 AGM60P90D, U1 URB2405S-6WR3

Commit message: Address design review R1: INA236, J15 polarity, review fixes
M1: U2-U5 are now TI INA236AIDDFR (C5443912, 50 V abs max, TSOT-23-8)
instead of the INA226 (40 V), since the SMBJ30A clamps at up to 48.4 V.
A project INA236 symbol keeps the INA226 body so the Flasher relay
wiring lands on the same pins; A1 and VBUS are gone (bus read on IN-),
addresses 0x40-0x43 via A0 = GND / VS / SDA / SCL. Same CONFIG / CAL /
MASK / ALERT values; notes give the 1.6 mV bus LSB and Device ID.
M3: J15 servo 24 V is pin 1 = +24 V like every power terminal.
L4: R38 servo RX series resistor 1k (limits PA3 back-feed).
L2: "current present" threshold 3 mA. L6: Power notes use 13 A / 2.2 W.
M2 / L5: silkscreen notes for "5V LOAD CELL - NEVER 24V" and
"CAN - NOT ETHERNET" (no keyed connector, by choice).
RJ45 1x4 footprint rebuilt from the HCTL drawing (14.0 mm ports,
Ø1.5 shield and Ø3.2 peg positions); U1 / U9 / U10 checked against the
JLC library and YLPTEC drawing. HANDOFF gains the review status table
and a layout checklist.

Co-Authored-By: Claude Opus 5.5 <noreply@anthropic.com>
Other:
- note added: "GND_24V: 24 V return (XT30 pin 2, relay outputs, sensor 0 V, TVS, bulk caps, DC/DC input side). GND: logic (module, INA236, ADS1232, DC/DC output). NT1: the only joint between them (the INA236s measure +24V against GND). Place it at the DC/DC."
- note added: "J5 XT30 (as on the MES4-Flasher): pin 1 + flat end, pin 2 - chamfered end. F1 15A fast fuse (Nano2 2410, 65 V): protects the XT30 and the board copper; a realistic 6-8 A stays under its 75 % derating (11 A); all loads at their limit (≈ 13 A, see the budget) would not. Each relay output has its own 3 A PTC, so a load short never blows F1. Q1 P-MOSFET reverse-polarity block: correct polarity turns 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"
- note added: "L1 10 µH + C4 / C5, with C2 on +24V: pi filter in front of the DC/DC only. Relay contacts, INA236s and sensors use the unfiltered +24V. U1 URB2405S-6WR3 (as on the MES4-Flasher): 9-36 V in, 5 V 1.2 A, short-circuit protected. CTRL open = on. C5 = the maker's 100 µF input cap; C6 / C7 = output caps. The maker's EMC circuit adds a 470 µH common-mode choke + 1 nF Y caps: not fitted, because NT1 ties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"
- note removed: "GND_24V: 24 V return (XT30 pin 2, relay outputs, sensor 0 V, TVS, bulk caps, DC/DC input side). GND: logic (module, INA226, ADS1232, DC/DC output). NT1: the only joint between them (the INA226s measure +24V against GND). Place it at the DC/DC."
- note removed: "J5 XT30 (as on the MES4-Flasher): pin 1 + flat end, pin 2 - chamfered end. F1 15A fast fuse (Nano2 2410, 65 V): protects the XT30 and the board copper; the 8.5 A worst case stays under its 75 % derating. Each relay output has its own 3 A PTC, so a load short never blows F1. Q1 P-MOSFET reverse-polarity block: correct polarity turns it on (Vgs clamped by D8, R6 10k to GND_24V); a reversed lead lea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"
- note removed: "L1 10 µH + C4 / C5, with C2 on +24V: pi filter in front of the DC/DC only. Relay contacts, INA226s and sensors use the unfiltered +24V. U1 URB2405S-6WR3 (as on the MES4-Flasher): 9-36 V in, 5 V 1.2 A, short-circuit protected. CTRL open = on. C5 = the maker's 100 µF input cap; C6 / C7 = output caps. The maker's EMC circuit adds a 470 µH common-mode choke + 1 nF Y caps: not fitted, because NT1 ties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"

Commit message: Add whole-board LTspice simulations, IMU notes and the R2 review package
sim/: 16 LTspice benches grouped by schematic sheet (Power, Relays,
Sensors, LoadCell, AuxPower, IMU, Winch, Main) on the real supply chain
(DDR-480C-24 at 24 V and a 24 V Li-ion pack via XY-CD63L, diode-OR'd by
an Autoro AB20). run_sims.py runs them, make_report.py builds
report.html. All pass; the IEC 0.5 kV surge is not applicable to this
internal, isolated supply. Raw waveforms and logs are git-ignored.

IMU: 3DM-CV7-AHRS on the C-Series Connectivity Board (6212-3009). The
AuxPower and Main notes, README and HANDOFF now say J14's 9 V goes to the
board's Vaux only (never Vpri), not together with the USB cable; the
power budget uses the real ~0.02 A at 24 V.

review/: MES4-Carrier-EC_Review-Package_R2.pdf, 26 pages: changes since
R1, status of every R1 finding, open items, the simulation report and
the regenerated 11-page schematic. HANDOFF records the supply chain and
the M4 results.

Co-Authored-By: Claude Opus 5.5 <noreply@anthropic.com>
Other:
- note added: "24 V current: relays ≤ 4 × 2 A (CIF §7; realistic 3-5 A: lamp ~0.3 A, DRL, 1.5 A solenoid), sensors 2 × ≤ 100 mA, logic DC/DC ≈ 0.15 A, IMU 9 V ≈ 0.02 A (CV7 0.23 W) + screen 5 V ≤ 0.95 A + door servo ≤ 3 A (page 9). Realistic total ≈ 6-8 A. Every load at its limit at once (≈ 13 A) would exceed F1 15A's 75 % derating (11 A) and the XT30's 15 A rating: don't stall the servo while all four relays c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"
- note removed: "24 V current: relays ≤ 4 × 2 A (CIF §7; realistic 3-5 A: lamp ~0.3 A, DRL, 1.5 A solenoid), sensors 2 × ≤ 100 mA, logic DC/DC ≈ 0.15 A, IMU 9 V ≤ 0.5 A + screen 5 V ≤ 0.95 A + door servo ≤ 3 A (page 9). Realistic total ≈ 6-8 A. Every load at its limit at once (≈ 13 A) would exceed F1 15A's 75 % derating (11 A) and the XT30's 15 A rating: don't stall the servo while all four relays carry 2 A. Nois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"
Changed lines of the file:
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@@
 		(effects (font (size 2 2) (bold yes)) (justify left top))
 	)
-	(text "24 V current: relays ≤ 4 × 2 A (CIF §7; realistic 3-5 A: lamp ~0.3 A, DRL, 1.5 A solenoid), sensors\n2 × ≤ 100 mA, logic DC/DC ≈ 0.15 A, IMU 9 V ≤ 0.5 A + screen 5 V ≤ 0.95 A + door servo ≤ 3 A (page 9).\nRealistic total ≈ 6-8 A. Every load at its limit at once (≈ 13 A) would exceed F1 15A's 75 % derating\n(11 A) and the XT30's 15 A rating: don't stall the servo while all four relays carry 2 A.\n\nNoise and transients, from the cable inwards:\n1. D9 SMBJ30A clamps surges and inductive spikes on the 24 V bus.\n2. C1 electrolytic damps the cable LC: no ringing above 24 V on hot-plug.\n3. C2 / C3 ceramics: low impedance for HF at the input.\n4. Pi filter C2 + L1 + C4 / C5 feeds only the DC/DC: the logic supply is decoupled\n   from the bus, and the converter's switching noise stays off it.\n5. Isolated DC/DC: the grounds meet only at NT1, so relay load currents never flow in GND.\n6. Pi filter F2 + FB1 + C8 / C9 on the module 5 V, and FB2 again on the ADS1232 AVDD.\n7. Flyback diodes at every relay coil (1N4148W) and every output (SS34).\n8. Sensor supplies: 100 mA PTC + 100 nF / 50 V at each terminal."
+	(text "24 V current: relays ≤ 4 × 2 A (CIF §7; realistic 3-5 A: lamp ~0.3 A, DRL, 1.5 A solenoid), sensors\n2 × ≤ 100 mA, logic DC/DC ≈ 0.15 A, IMU 9 V ≈ 0.02 A (CV7 0.23 W) + screen 5 V ≤ 0.95 A + door servo ≤ 3 A (page 9).\nRealistic total ≈ 6-8 A. Every load at its limit at once (≈ 13 A) would exceed F1 15A's 75 % derating\n(11 A) and the XT30's 15 A rating: don't stall the servo while all four relays carry 2 A.\n\nNoise and transients, from the cable inwards:\n1. D9 SMBJ30A clamps surges and inductive spikes on the 24 V bus.\n2. C1 electrolytic damps the cable LC: no ringing above 24 V on hot-plug.\n3. C2 / C3 ceramics: low impedance for HF at the input.\n4. Pi filter C2 + L1 + C4 / C5 feeds only the DC/DC: the logic supply is decoupled\n   from the bus, and the converter's switching noise stays off it.\n5. Isolated DC/DC: the grounds meet only at NT1, so relay load currents never flow in GND.\n6. Pi filter F2 + FB1 + C8 / C9 on the module 5 V, and FB2 again on the ADS1232 AVDD.\n7. Flyback diodes at every relay coil (1N4148W) and every output (SS34).\n8. Sensor supplies: 100 mA PTC + 100 nF / 50 V at each terminal."
 		(exclude_from_sim no)
 		(at 200.66 27.94 0)

Commit message: One ground and a 4-layer board
- GND_24V merged into GND (ONE_GND in gen.py): every GND_24V power symbol
  becomes GND, net tie NT1 left out, notes reworded. Symbol UUIDs unchanged,
  so every footprint keeps its link.
- 4 layers, JLC04161H-7628 stackup (1.6 mm, ENIG): Top Signal / GND plane
  (In1) / +24V plane (In2) / Bottom Signal.
- Net classes: Out_3A (1.5 mm) for +24V_SRV, +5V_SCR, VBUS_SCR; +24V_AUX to
  24V_Power; +5V_SRV, +9V_IMU, IMU_9V to Power; INA236 shunt pattern fixed
  (Net-(U*-IN-)).
- J1's NPTH holes back to F&B.Cu as in its library footprint.

ERC 0, checks passed, DRC 11 silkscreen warnings, schematic parity clean.

Co-Authored-By: Claude Opus 5.5 <noreply@anthropic.com>
Parts:
- removed NT1: NetTie, NetTie:NetTie-2_SMD_Pad2.0mm, symbol Device:NetTie_2
- TP7: value GND_24V -> GND
Connections:
- net GND_24V is gone; now on net GND: C1.2, C2.2, C3.2, C4.2, C5.2, D9.2 (A), J5.2 (Pin_2), LED3.1 (K), R6.2, TP7.1, U1.1 (GND)
Other:
- note added: "2 mm pads with a 1 mm hole: probe tip, or solder a wire loop for clips (not in the BOM). Clip the scope ground to either GND pad, the one nearer the circuit you probe."
- note added: "L1 10 µH + C4 / C5, with C2 on +24V: pi filter in front of the DC/DC only. Relay contacts, INA236s and sensors use the unfiltered +24V. U1 URB2405S-6WR3 (as on the MES4-Flasher): 9-36 V in, 5 V 1.2 A, short-circuit protected. CTRL open = on. C5 = the maker's 100 µF input cap; C6 / C7 = output caps. The maker's EMC circuit adds a 470 µH common-mode choke + 1 nF Y caps: not fitted, because One GND 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"
- note added: "One ground, GND, for the 24 V side and the logic: XT30 pin 2, relay outputs, sensor 0 V, TVS, bulk caps, both DC/DC sides, module, INA236, ADS1232. PCB: a solid GND plane on In1.Cu under the whole board."
- note removed: "2 mm pads with a 1 mm hole: probe tip, or solder a wire loop for clips (not in the BOM). Clip the scope ground to GND for the module side and to GND_24V for the 24 V side."
- note removed: "GND_24V: 24 V return (XT30 pin 2, relay outputs, sensor 0 V, TVS, bulk caps, DC/DC input side). GND: logic (module, INA236, ADS1232, DC/DC output). NT1: the only joint between them (the INA236s measure +24V against GND). Place it at the DC/DC."
- note removed: "L1 10 µH + C4 / C5, with C2 on +24V: pi filter in front of the DC/DC only. Relay contacts, INA236s and sensors use the unfiltered +24V. U1 URB2405S-6WR3 (as on the MES4-Flasher): 9-36 V in, 5 V 1.2 A, short-circuit protected. CTRL open = on. C5 = the maker's 100 µF input cap; C6 / C7 = output caps. The maker's EMC circuit adds a 470 µH common-mode choke + 1 nF Y caps: not fitted, because NT1 ties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"

Commit message: Placement and silkscreen pass: ADS by the load-cell inputs, test points, logo
- Left column top to bottom: ADS1232 under J12/J13 (input filter toward the
  connectors), STDC14 + ESD grid, then the MES4-MCU slot moved down 22.3 mm;
  RESET (SW1) beside J1 with the 5 V socket caps C8/C9.
- Test points named by what they feed (TP_NAME in gen.py: 24V, 24V FILT,
  5V MAIN, 5V MCU, 3V3, 9V IMU, 5V SCREEN); bottom row in a Flasher-style
  rounded box, 24V/GND under the XT30, 5V SCREEN/GND by the screen USB-C.
- Supply LEDs centred between SW2 and the winch block; short knockout labels
  all one box size (drawn as cut-out silk shapes).
- + at the anode of every two-pin diode and LED; SW2 marked IMU PWR with
  OFF/ON (slider toward pin 1 = on); mounting-hole refs off the silkscreen.
- Sensor inputs in the column under L1/L2, U10 output caps against U10,
  servo support parts in the square by J17, FE-URT-2 J17/J15 label boxes,
  Monkey Robotics logo (43 x 9.3 mm) in the freed space.

ERC 0, DRC 14 silkscreen warnings (13 edge, J1 circle), schematic parity clean.

Co-Authored-By: Claude Opus 5.5 <noreply@anthropic.com>
Parts:
- TP1: value +24V -> 24V
- TP2: value +24V_DC -> 24V FILT
- TP3: value +5V_24 -> 5V MAIN
- TP4: value +5V -> 5V MCU
- TP5: value +3V3_MOD -> 3V3
Changed lines of the file:
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@@
 			(effects (font (size 1.27 1.27)) (justify right))
 		)
-		(property "Value" "+24V"
+		(property "Value" "24V"
 			(at 29.21 209.55 0)
 			(effects (font (size 1.27 1.27)) (justify right))
@@
 			(effects (font (size 1.27 1.27)) (justify right))
 		)
-		(property "Value" "+24V_DC"
+		(property "Value" "24V FILT"
 			(at 57.15 209.55 0)
 			(effects (font (size 1.27 1.27)) (justify right))
@@
 			(effects (font (size 1.27 1.27)) (justify right))
 		)
-		(property "Value" "+5V_24"
+		(property "Value" "5V MAIN"
 			(at 85.09 209.55 0)
 			(effects (font (size 1.27 1.27)) (justify right))
@@
 			(effects (font (size 1.27 1.27)) (justify right))
 		)
-		(property "Value" "+5V"
+		(property "Value" "5V MCU"
 			(at 113.03 209.55 0)
 			(effects (font (size 1.27 1.27)) (justify right))
@@
 			(effects (font (size 1.27 1.27)) (justify right))
 		)
-		(property "Value" "+3V3_MOD"
+		(property "Value" "3V3"
 			(at 140.97 209.55 0)
 			(effects (font (size 1.27 1.27)) (justify right))
