File: MES4_Carrier_EC/Power.kicad_sch (KiCad schematic)
At the start: 28 parts, among them J5 24V IN, Q1 AGM60P90D, U1 URB2405S-6WR3

Commit message: Fix design review R3 findings: U9 part, stale LCSC fields, labels, J16
- B1: U9 is now YLPTEC URB2409S-6WR3 (C7468814, 9 V 6 W) on U1's
  footprint; the 10 W URB2409S-10WR3 isn't in JLC's assembly library.
  The production BOM had a 5 V module at U9 and the wrong SW2 because
  EasyEDA footprints carry an "LCSC Part" field the Fabrication Toolkit
  reads first: libs.py strips it (and the unprintable pin-1 dots it was
  copying back), and the new parts_sync.py syncs board footprints,
  values, fields and BOM flags from the schematic. TP1-TP9 and H2-H5
  are out of the BOM and CPL.
- M2 / L5: "5V LOAD CELL" across J12 / J13; "CANBUS" knockout by J4.
- B2: J16 moves 1.25 mm west so its mouth reaches the board edge.
- B8 / N6: README (one ground, U9, J16, labels, TPs), schematic notes
  and HANDOFF updated; 1:1 A4 print refreshed.
- DRC with parity at the 3 accepted J4 notes; nets, audit, DFM clean.
  production/ is stale until the Fabrication Toolkit is re-run.

Co-Authored-By: Claude Opus 5.5 <noreply@anthropic.com>
Parts:
- TP1, TP2, TP3, TP4, TP5, TP6, TP7: now left out of the parts list
Changed lines of the file:
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@@
 		(unit 1)
 		(exclude_from_sim no)
-		(in_bom yes)
+		(in_bom no)
 		(on_board yes)
 		(dnp no)
@@
 		(unit 1)
 		(exclude_from_sim no)
-		(in_bom yes)
+		(in_bom no)
 		(on_board yes)
 		(dnp no)
@@
 		(unit 1)
 		(exclude_from_sim no)
-		(in_bom yes)
+		(in_bom no)
 		(on_board yes)
 		(dnp no)
@@
 		(unit 1)
 		(exclude_from_sim no)
-		(in_bom yes)
+		(in_bom no)
 		(on_board yes)
 		(dnp no)
@@
 		(unit 1)
 		(exclude_from_sim no)
-		(in_bom yes)
+		(in_bom no)
 		(on_board yes)
 		(dnp no)
@@
 		(unit 1)
 		(exclude_from_sim no)
-		(in_bom yes)
+		(in_bom no)
 		(on_board yes)
 		(dnp no)
@@
 		(unit 1)
 		(exclude_from_sim no)
-		(in_bom yes)
-		(on_board yes)
-		(dnp no)
+		(in_bom no)
+		(on_board yes)
+		(dnp no)

Commit message: Check CPL rotations against JLC's footprints; fix Q1, K1-K4, J5
- cpl_check.py: fetches each LCSC part's EasyEDA footprint, matches
  pads (polarity names, numbers or shape), fits the rotation / offset
  JLC needs and compares with production/positions.csv.
- Q1 (TO-252) needs +180 deg and -1.8 mm, K1-K4 (SRD relays) +180 deg,
  J5 (XT30) +9.7 mm: set as Fabrication Toolkit FT Rotation / Position
  Offset fields on the symbols (gen.py, parts.py), copied to the board
  by parts_sync.py.
- production/ regenerated with the toolkit CLI: 169 of 181 placements
  match JLC; C1 / C5 / C27 (no JLC footprint) to check in the preview.
- HANDOFF updated.

Co-Authored-By: Claude Opus 5.5 <noreply@anthropic.com>
Parts:
- J5: FT Position Offset (none) -> 0,9.7
- Q1: FT Position Offset (none) -> -1.8,0; FT Rotation Offset (none) -> 180
Changed lines of the file:
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@@
+			(effects (font (size 1.27 1.27)) (hide yes))
+		)
+		(property "FT Position Offset" "0,9.7"
+			(at 25.4 50.8 0)
 			(effects (font (size 1.27 1.27)) (hide yes))
 		)
@@
 			(at 71.12 53.34 0)
 			(effects (font (size 1.27 1.27)) (hide yes))
+		)
+		(property "FT Rotation Offset" "180"
+			(at 71.12 53.34 0)
+			(effects (font (size 1.27 1.27)) (hide yes))
+		)
+		(property "FT Position Offset" "-1.8,0"
+			(at 71.12 53.34 0)
+			(effects (font (size 1.27 1.27)) (hide yes))

Commit message: Fix design review R4 (CPL), add 3D models, STEP and the enclosure
Review R4:
- E1 (blocking): the Fabrication Toolkit turns every CP_Elec 180 deg, but
  JLC's footprints for C1/C5/C27/C28/C30/C32/C38 have + on the same side
  as ours, so all seven would have been fitted reversed. gen.py now sets
  FT Rotation Offset 180 on every CP_Elec part (the toolkit adds it to its
  own 180), so the CPL keeps the board rotation.
- E2: J5's FT Position Offset 0,9.7 put the XT30 10 mm off; JLC's origin
  is ours. Removed; parts_sync.py now drops FT fields the schematic no
  longer has.
- E3: parts_sync.py keeps H2-H5's empty LCSC field (KiCad 10 field parity).
- cpl_check.py rewritten as a gate: places JLC's own footprint where the
  CPL says, every JLC pad must land on our pads (pegs included), pin n on
  our pin n wherever the pattern also fits at another turn; only
  non-polar two-pad parts may sit 180 deg round. 177/181 pass, 0 to fix.
- production.sh: Fabrication Toolkit CLI, then the gate; deletes the
  order zip if it fails. production/ regenerated through it.

3D / STEP: EasyEDA STEP models placed onto their pads (J1 M.2, J16, K5/K6,
U1/U9, SW2), LCSC STEPs for the KF250 terminals and fuses, standoffs
converted from VRML (wrl2step.py); review/MES4_Carrier_EC.step.

Enclosure: two-part FDM box generated from the board (FreeCAD): M3
heat-set inserts, connector openings, LED light guides and labels, M5
side tabs, engraved logo, P1S tolerances, no supports. The 82 MB
assembly STEP is regenerated, not committed.

Co-Authored-By: Claude Opus 5.5 <noreply@anthropic.com>
Parts:
- C1, C5: FT Rotation Offset (none) -> 180
- F1: footprint Fuse:Fuse_Littelfuse-NANO2-451_453 -> MES4-Carrier-EC:Fuse_Littelfuse-NANO2-451_453
- J5: FT Position Offset 0,9.7 -> (none)
Changed lines of the file:
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@@
-			(effects (font (size 1.27 1.27)) (hide yes))
-		)
-		(property "FT Position Offset" "0,9.7"
-			(at 25.4 50.8 0)
 			(effects (font (size 1.27 1.27)) (hide yes))
 		)
@@
 			(effects (font (size 1.27 1.27)))
 		)
-		(property "Footprint" "Fuse:Fuse_Littelfuse-NANO2-451_453"
+		(property "Footprint" "MES4-Carrier-EC:Fuse_Littelfuse-NANO2-451_453"
 			(at 50.8 50.8 0)
 			(effects (font (size 1.27 1.27)) (hide yes))
@@
 			(effects (font (size 1.27 1.27)) (hide yes))
 		)
+		(property "FT Rotation Offset" "180"
+			(at 116.84 54.61 0)
+			(effects (font (size 1.27 1.27)) (hide yes))
+		)
 		(pin "1"
 		)
@@
 			(at 71.12 140.97 0)
 			(effects (font (size 1.27 1.27)) (hide yes))
+		)
+		(property "FT Rotation Offset" "180"
+			(at 71.12 140.97 0)
+			(effects (font (size 1.27 1.27)) (hide yes))
