File: MES4_Carrier_EC/MES4_Carrier_EC.kicad_sch (KiCad schematic)
At the start: 0 parts

Commit message: Put relay coil feedback back on PA0-PA3 (MES4 GPIO standard)
All 14 module GPIOs now follow the MES4-CIF §2c table. The TCA9535 is
removed from the Relays 3-4 sheet and J1 fingers 43/45/47/49 drive the
relay 1-4 feedback dividers again. The winch relays are left undriven
(gate inputs no-connected, 100k pull-downs hold them off) until they
move to the TCA9535 + photoMOS design (HANDOFF.md step 2).

Removing U4 renumbers U5-U12 to U4-U11 and C15-C45 to C14-C44; the
README refs follow. Adds generator/checks.py (pin/pad, single-pin nets,
duplicate UUIDs, LCSC numbers), run by run.sh after ERC.

Co-Authored-By: Claude Opus 5.5 <noreply@anthropic.com>
Other:
- note added: "1 safety light: PA8 drive, PA0 FB, INA226 0x40 2 LED DRL: PC6 drive, PA1 FB, 0x41 3 battery stopper: PB3 drive, PA2 FB, 0x44 4 spare: PA7 drive, PA3 FB, 0x45 GPIO → 100 Ω → AO3400A → 5 V coil (SRD-5VDC-SL-A, on +5V_24). +24V → 30 mΩ shunt → contact → 3A PTC → output (2 A continuous). Coil feedback 10k / 15k → PA0-PA3. INA226 per channel: load current + 24 V rail, ALERT → PA15."
- note added: "E-Crawler carrier for one MES4-MCU module (MES4-CIF rev A-d6). Circuits taken from the MES4-Flasher: PC817 sensor inputs, ADS1232 load cell, relay channels (driver, coil feedback, INA226) and the XT30 / URB2405S 24 V input. GPIO budget: 4 relay drives + 4 coil feedbacks + ALERT + 3 ADS1232 + 2 sensors = 14, as in the MES4-CIF §2c table. Servo UART (SC16IS740) and, next, the winch (TCA9535) run on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"
- note added: "Load cell (U8 ADS1232)"
- note added: "Own L pi filter from +24V. U9 URB2409S-10WR3 → 9 V → SW2 switch → J14 IMU terminal (as on the MES3.1 carrier). U10 URB2405LD-20WR3 → 5 V 4 A → 3 A PTC → J16 USB-C (Rp 10k: 5 V / 3 A) → ARZOPA Z1C screen. Door servo (FE-URT-2): J15 24 V + J17 UART via the I²C bridge."
- note added: "Two IM03GR relays, as on the MES2_Extension (AO3400A drivers). TODO: drive from a TCA9535 on I²C1 (PA0 / PA1 are coil FB). Contacts switch the 48 V winch controller's direction inputs. Hardware interlock: both on = both open."
- note added: "coil FB PA0-PA3"
- note removed: "1 safety light: PA8 drive, PA0 FB, INA226 0x40 2 LED DRL: PC6 drive, PA1 FB, 0x41 3 battery stopper: PB3 drive, PA2 FB, 0x44 4 spare: PA7 drive, PA3 FB, 0x45 GPIO → 100 Ω → AO3400A → 5 V coil (SRD-5VDC-SL-A, on +5V_24). +24V → 30 mΩ shunt → contact → 3A PTC → output (2 A continuous). Coil feedback 10k / 15k → TCA9535 (I²C). INA226 per channel: load current + 24 V rail, ALERT → PA15."
- note removed: "E-Crawler carrier for one MES4-MCU module (MES4-CIF rev A-d6). Circuits taken from the MES4-Flasher: PC817 sensor inputs, ADS1232 load cell, relay channels (driver, coil feedback, INA226) and the XT30 / URB2405S 24 V input. GPIO budget: 4 relay drives + ALERT + 3 ADS1232 + 2 sensors + winch (2) = 12; PA2 / PA3 free (servo on the I²C bridge). Relay coil feedback goes through a TCA9535 I²C expander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"
- note removed: "Load cell (U9 ADS1232)"
- note removed: "Own L pi filter from +24V. U10 URB2409S-10WR3 → 9 V → SW2 switch → J14 IMU terminal (as on the MES3.1 carrier). U11 URB2405LD-20WR3 → 5 V 4 A → 3 A PTC → J16 USB-C (Rp 10k: 5 V / 3 A) → ARZOPA Z1C screen. Door servo (FE-URT-2): J15 24 V + J17 UART via the I²C bridge."
- note removed: "Two IM03GR relays, as on the MES2_Extension: PA0 → CLK, PA1 → ACLK (AO3400A drivers). Contacts switch the 48 V winch controller's direction inputs. Hardware interlock: both on = both open."
- note removed: "coil FB (I²C)"
Changed lines of the file:
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@@
 		(effects (font (size 2.2 2.2) (bold yes)) (justify left top))
 	)
-	(text "1 safety light: PA8 drive, PA0 FB, INA226 0x40\n2 LED DRL: PC6 drive, PA1 FB, 0x41\n3 battery stopper: PB3 drive, PA2 FB, 0x44\n4 spare: PA7 drive, PA3 FB, 0x45\n\nGPIO → 100 Ω → AO3400A → 5 V coil\n(SRD-5VDC-SL-A, on +5V_24).\n+24V → 30 mΩ shunt → contact →\n3A PTC → output (2 A continuous).\nCoil feedback 10k / 15k → TCA9535 (I²C).\nINA226 per channel: load current +\n24 V rail, ALERT → PA15."
+	(text "1 safety light: PA8 drive, PA0 FB, INA226 0x40\n2 LED DRL: PC6 drive, PA1 FB, 0x41\n3 battery stopper: PB3 drive, PA2 FB, 0x44\n4 spare: PA7 drive, PA3 FB, 0x45\n\nGPIO → 100 Ω → AO3400A → 5 V coil\n(SRD-5VDC-SL-A, on +5V_24).\n+24V → 30 mΩ shunt → contact →\n3A PTC → output (2 A continuous).\nCoil feedback 10k / 15k → PA0-PA3.\nINA226 per channel: load current +\n24 V rail, ALERT → PA15."
 		(exclude_from_sim no)
 		(at 208.28 48.26 0)
@@
 		(fill (type color) (color 238 228 250 1))
 	)
-	(text "Load cell (U9 ADS1232)"
+	(text "Load cell (U8 ADS1232)"
 		(exclude_from_sim no)
 		(at 208.28 159.77 0)
@@
 		(effects (font (size 2.2 2.2) (bold yes)) (justify left top))
 	)
-	(text "Own L pi filter from +24V.\nU10 URB2409S-10WR3 → 9 V →\nSW2 switch → J14 IMU terminal\n(as on the MES3.1 carrier).\nU11 URB2405LD-20WR3 → 5 V 4 A\n→ 3 A PTC → J16 USB-C (Rp 10k:\n5 V / 3 A) → ARZOPA Z1C screen.\nDoor servo (FE-URT-2): J15 24 V\n+ J17 UART via the I²C bridge."
+	(text "Own L pi filter from +24V.\nU9 URB2409S-10WR3 → 9 V →\nSW2 switch → J14 IMU terminal\n(as on the MES3.1 carrier).\nU10 URB2405LD-20WR3 → 5 V 4 A\n→ 3 A PTC → J16 USB-C (Rp 10k:\n5 V / 3 A) → ARZOPA Z1C screen.\nDoor servo (FE-URT-2): J15 24 V\n+ J17 UART via the I²C bridge."
 		(exclude_from_sim no)
 		(at 312.42 149.86 0)
@@
 		(effects (font (size 2.2 2.2) (bold yes)) (justify left top))
 	)
-	(text "Two IM03GR relays, as on the\nMES2_Extension: PA0 → CLK,\nPA1 → ACLK (AO3400A drivers).\nContacts switch the 48 V winch\ncontroller's direction inputs.\nHardware interlock: both on =\nboth open."
+	(text "Two IM03GR relays, as on the\nMES2_Extension (AO3400A drivers).\nTODO: drive from a TCA9535 on\nI²C1 (PA0 / PA1 are coil FB).\nContacts switch the 48 V winch\ncontroller's direction inputs.\nHardware interlock: both on =\nboth open."
 		(exclude_from_sim no)
 		(at 312.42 48.26 0)
@@
 		(fill (type color) (color 30 80 200 1))
 	)
-	(text "coil FB (I²C)"
-		(exclude_from_sim no)
-		(at 185.42 77.47 0)
+	(text "coil FB\nPA0-PA3"
+		(exclude_from_sim no)
+		(at 185.42 74.93 0)
 		(effects (font (size 1.6 1.6) (color 30 80 200 1)) (justify left top))
 	)
@@
 		(effects (font (size 2.2 2.2) (bold yes)) (justify left top))
 	)
-	(text "E-Crawler carrier for one MES4-MCU module (MES4-CIF rev A-d6). Circuits taken from the MES4-Flasher: PC817 sensor inputs,\nADS1232 load cell, relay channels (driver, coil feedback, INA226) and the XT30 / URB2405S 24 V input.\nGPIO budget: 4 relay drives + ALERT + 3 ADS1232 + 2 sensors + winch (2) = 12; PA2 / PA3 free (servo on the I²C bridge).\nRelay coil feedback goes through a TCA9535 I²C expander (MES4-CIF §7c).\nRelay drive per CIF §7a (AO3400A, 100 Ω, 100k pull-down); the Flasher uses a 2SC2884 BJT for the same job.\nNo hot-plug: unplug the 24 V XT30 before inserting or removing the module.\nPages: Main (2), CAN (3), Power (4), Relays 1-2 (5), Relays 3-4 (6), Sensors (7), LoadCell (8), AuxPower (9), Winch (10)."
+	(text "E-Crawler carrier for one MES4-MCU module (MES4-CIF rev A-d6). Circuits taken from the MES4-Flasher: PC817 sensor inputs,\nADS1232 load cell, relay channels (driver, coil feedback, INA226) and the XT30 / URB2405S 24 V input.\nGPIO budget: 4 relay drives + 4 coil feedbacks + ALERT + 3 ADS1232 + 2 sensors = 14, as in the MES4-CIF §2c table.\nServo UART (SC16IS740) and, next, the winch (TCA9535) run on I²C1, so they need no module pins.\nRelay drive per CIF §7a (AO3400A, 100 Ω, 100k pull-down); the Flasher uses a 2SC2884 BJT for the same job.\nNo hot-plug: unplug the 24 V XT30 before inserting or removing the module.\nPages: Main (2), CAN (3), Power (4), Relays 1-2 (5), Relays 3-4 (6), Sensors (7), LoadCell (8), AuxPower (9), Winch (10)."
 		(exclude_from_sim no)
 		(at 20.32 221 0)
@@
 		(instances
 			(project "MES4_Carrier_EC"
-				(path "/b63007a2-51a5-5afa-ba23-67ba50ea48db"
+				(path "/86b406aa-a59b-5773-8968-b904bb1c5afe"
 					(page "2")
 				)
@@
 		(instances
 			(project "MES4_Carrier_EC"
-				(path "/b63007a2-51a5-5afa-ba23-67ba50ea48db"
+				(path "/86b406aa-a59b-5773-8968-b904bb1c5afe"
 					(page "3")
 				)
@@
 		(instances
 			(project "MES4_Carrier_EC"
-				(path "/b63007a2-51a5-5afa-ba23-67ba50ea48db"
+				(path "/86b406aa-a59b-5773-8968-b904bb1c5afe"
 					(page "4")
 				)
@@
 		(instances
 			(project "MES4_Carrier_EC"
-				(path "/b63007a2-51a5-5afa-ba23-67ba50ea48db"
+				(path "/86b406aa-a59b-5773-8968-b904bb1c5afe"
 					(page "5")
 				)
@@
 		(instances
 			(project "MES4_Carrier_EC"
-				(path "/b63007a2-51a5-5afa-ba23-67ba50ea48db"
+				(path "/86b406aa-a59b-5773-8968-b904bb1c5afe"
 					(page "6")
 				)
@@
 		(instances
 			(project "MES4_Carrier_EC"
-				(path "/b63007a2-51a5-5afa-ba23-67ba50ea48db"
+				(path "/86b406aa-a59b-5773-8968-b904bb1c5afe"
 					(page "7")
 				)
@@
 		(instances
 			(project "MES4_Carrier_EC"
-				(path "/b63007a2-51a5-5afa-ba23-67ba50ea48db"
+				(path "/86b406aa-a59b-5773-8968-b904bb1c5afe"
 					(page "8")
 				)
@@
 		(instances
 			(project "MES4_Carrier_EC"
-				(path "/b63007a2-51a5-5afa-ba23-67ba50ea48db"
+				(path "/86b406aa-a59b-5773-8968-b904bb1c5afe"
 					(page "9")
 				)
@@
 		(instances
 			(project "MES4_Carrier_EC"
-				(path "/b63007a2-51a5-5afa-ba23-67ba50ea48db"
+				(path "/86b406aa-a59b-5773-8968-b904bb1c5afe"
 					(page "10")
 				)

Commit message: Drop relay coil feedback; winch on PA0/PA1, servo on USART2
User decision: free the four feedback pins instead of adding an I²C
expander. The Flasher template's 10k/15k/10 nF dividers are removed from
all relay channels and relay diagnosis is INA226-only. PA0/PA1 drive the
IM03GR winch relays again and PA2/PA3 carry the door servo UART
(USART2), so the SC16IS740 bridge, its crystal and caps, and the unused
TCA9535 code are removed. This deliberately differs from the MES4-CIF
§2c GPIO table; the GPIO map, root notes, README and HANDOFF say so.

189 parts, ERC clean, checks.py passes. README refs follow the
renumbering.

Co-Authored-By: Claude Opus 5.5 <noreply@anthropic.com>
Other:
- note added: "1 safety light: PA8 drive, INA226 0x40 2 LED DRL: PC6 drive, INA226 0x41 3 battery stopper: PB3 drive, INA226 0x44 4 spare: PA7 drive, INA226 0x45 GPIO → 100 Ω → AO3400A → 5 V coil (SRD-5VDC-SL-A, on +5V_24). +24V → 30 mΩ shunt → contact → 3A PTC → output (2 A continuous). No coil feedback (pins used elsewhere). INA226 per channel: load current + 24 V rail, ALERT → PA15."
- note added: "E-Crawler carrier for one MES4-MCU module (MES4-CIF rev A-d6). Circuits taken from the MES4-Flasher: PC817 sensor inputs, ADS1232 load cell, relay channels (driver, INA226) and the XT30 / URB2405S 24 V input. GPIO budget: 4 relay drives + ALERT + 3 ADS1232 + 2 sensors + winch (2) + servo USART2 (2) = 14. Differs from the MES4-CIF §2c table: no relay coil feedback, so PA0-PA3 drive the winch and t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"
- note added: "Own L pi filter from +24V. U9 URB2409S-10WR3 → 9 V → SW2 switch → J14 IMU terminal (as on the MES3.1 carrier). U10 URB2405LD-20WR3 → 5 V 4 A → 3 A PTC → J16 USB-C (Rp 10k: 5 V / 3 A) → ARZOPA Z1C screen. Door servo (FE-URT-2): J15 24 V + J17 UART (USART2)."
- note added: "Two IM03GR relays, as on the MES2_Extension: PA0 → CLK, PA1 → ACLK (AO3400A drivers). Contacts switch the 48 V winch controller's direction inputs. Hardware interlock: both on = both open."
- note removed: "1 safety light: PA8 drive, PA0 FB, INA226 0x40 2 LED DRL: PC6 drive, PA1 FB, 0x41 3 battery stopper: PB3 drive, PA2 FB, 0x44 4 spare: PA7 drive, PA3 FB, 0x45 GPIO → 100 Ω → AO3400A → 5 V coil (SRD-5VDC-SL-A, on +5V_24). +24V → 30 mΩ shunt → contact → 3A PTC → output (2 A continuous). Coil feedback 10k / 15k → PA0-PA3. INA226 per channel: load current + 24 V rail, ALERT → PA15."
- note removed: "E-Crawler carrier for one MES4-MCU module (MES4-CIF rev A-d6). Circuits taken from the MES4-Flasher: PC817 sensor inputs, ADS1232 load cell, relay channels (driver, coil feedback, INA226) and the XT30 / URB2405S 24 V input. GPIO budget: 4 relay drives + 4 coil feedbacks + ALERT + 3 ADS1232 + 2 sensors = 14, as in the MES4-CIF §2c table. Servo UART (SC16IS740) and, next, the winch (TCA9535) run on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"
- note removed: "Own L pi filter from +24V. U9 URB2409S-10WR3 → 9 V → SW2 switch → J14 IMU terminal (as on the MES3.1 carrier). U10 URB2405LD-20WR3 → 5 V 4 A → 3 A PTC → J16 USB-C (Rp 10k: 5 V / 3 A) → ARZOPA Z1C screen. Door servo (FE-URT-2): J15 24 V + J17 UART via the I²C bridge."
- note removed: "Two IM03GR relays, as on the MES2_Extension (AO3400A drivers). TODO: drive from a TCA9535 on I²C1 (PA0 / PA1 are coil FB). Contacts switch the 48 V winch controller's direction inputs. Hardware interlock: both on = both open."
- note removed: "coil FB PA0-PA3"
Changed lines of the file:
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@@
 		(effects (font (size 2.2 2.2) (bold yes)) (justify left top))
 	)
-	(text "1 safety light: PA8 drive, PA0 FB, INA226 0x40\n2 LED DRL: PC6 drive, PA1 FB, 0x41\n3 battery stopper: PB3 drive, PA2 FB, 0x44\n4 spare: PA7 drive, PA3 FB, 0x45\n\nGPIO → 100 Ω → AO3400A → 5 V coil\n(SRD-5VDC-SL-A, on +5V_24).\n+24V → 30 mΩ shunt → contact →\n3A PTC → output (2 A continuous).\nCoil feedback 10k / 15k → PA0-PA3.\nINA226 per channel: load current +\n24 V rail, ALERT → PA15."
+	(text "1 safety light: PA8 drive, INA226 0x40\n2 LED DRL: PC6 drive, INA226 0x41\n3 battery stopper: PB3 drive, INA226 0x44\n4 spare: PA7 drive, INA226 0x45\n\nGPIO → 100 Ω → AO3400A → 5 V coil\n(SRD-5VDC-SL-A, on +5V_24).\n+24V → 30 mΩ shunt → contact →\n3A PTC → output (2 A continuous).\nNo coil feedback (pins used elsewhere).\nINA226 per channel: load current +\n24 V rail, ALERT → PA15."
 		(exclude_from_sim no)
 		(at 208.28 48.26 0)
@@
 		(effects (font (size 2.2 2.2) (bold yes)) (justify left top))
 	)
-	(text "Own L pi filter from +24V.\nU9 URB2409S-10WR3 → 9 V →\nSW2 switch → J14 IMU terminal\n(as on the MES3.1 carrier).\nU10 URB2405LD-20WR3 → 5 V 4 A\n→ 3 A PTC → J16 USB-C (Rp 10k:\n5 V / 3 A) → ARZOPA Z1C screen.\nDoor servo (FE-URT-2): J15 24 V\n+ J17 UART via the I²C bridge."
+	(text "Own L pi filter from +24V.\nU9 URB2409S-10WR3 → 9 V →\nSW2 switch → J14 IMU terminal\n(as on the MES3.1 carrier).\nU10 URB2405LD-20WR3 → 5 V 4 A\n→ 3 A PTC → J16 USB-C (Rp 10k:\n5 V / 3 A) → ARZOPA Z1C screen.\nDoor servo (FE-URT-2): J15 24 V\n+ J17 UART (USART2)."
 		(exclude_from_sim no)
 		(at 312.42 149.86 0)
@@
 		(effects (font (size 2.2 2.2) (bold yes)) (justify left top))
 	)
-	(text "Two IM03GR relays, as on the\nMES2_Extension (AO3400A drivers).\nTODO: drive from a TCA9535 on\nI²C1 (PA0 / PA1 are coil FB).\nContacts switch the 48 V winch\ncontroller's direction inputs.\nHardware interlock: both on =\nboth open."
+	(text "Two IM03GR relays, as on the\nMES2_Extension: PA0 → CLK,\nPA1 → ACLK (AO3400A drivers).\nContacts switch the 48 V winch\ncontroller's direction inputs.\nHardware interlock: both on =\nboth open."
 		(exclude_from_sim no)
 		(at 312.42 48.26 0)
@@
 		(exclude_from_sim no)
 		(at 185.42 56.52 0)
-		(effects (font (size 1.6 1.6) (color 30 80 200 1)) (justify left top))
-	)
-	(polyline
-		(pts (xy 205.74 81.28) (xy 182.88 81.28))
-		(stroke (width 0.8) (type solid) (color 30 80 200 1))
-		(fill (type none))
-	)
-	(polyline
-		(pts (xy 182.88 81.28) (xy 185.68 80.18) (xy 185.68 82.38) (xy 182.88 81.28))
-		(stroke (width 0.1) (type solid) (color 30 80 200 1))
-		(fill (type color) (color 30 80 200 1))
-	)
-	(text "coil FB\nPA0-PA3"
-		(exclude_from_sim no)
-		(at 185.42 74.93 0)
 		(effects (font (size 1.6 1.6) (color 30 80 200 1)) (justify left top))
 	)
@@
 		(effects (font (size 2.2 2.2) (bold yes)) (justify left top))
 	)
-	(text "E-Crawler carrier for one MES4-MCU module (MES4-CIF rev A-d6). Circuits taken from the MES4-Flasher: PC817 sensor inputs,\nADS1232 load cell, relay channels (driver, coil feedback, INA226) and the XT30 / URB2405S 24 V input.\nGPIO budget: 4 relay drives + 4 coil feedbacks + ALERT + 3 ADS1232 + 2 sensors = 14, as in the MES4-CIF §2c table.\nServo UART (SC16IS740) and, next, the winch (TCA9535) run on I²C1, so they need no module pins.\nRelay drive per CIF §7a (AO3400A, 100 Ω, 100k pull-down); the Flasher uses a 2SC2884 BJT for the same job.\nNo hot-plug: unplug the 24 V XT30 before inserting or removing the module.\nPages: Main (2), CAN (3), Power (4), Relays 1-2 (5), Relays 3-4 (6), Sensors (7), LoadCell (8), AuxPower (9), Winch (10)."
+	(text "E-Crawler carrier for one MES4-MCU module (MES4-CIF rev A-d6). Circuits taken from the MES4-Flasher: PC817 sensor inputs,\nADS1232 load cell, relay channels (driver, INA226) and the XT30 / URB2405S 24 V input.\nGPIO budget: 4 relay drives + ALERT + 3 ADS1232 + 2 sensors + winch (2) + servo USART2 (2) = 14.\nDiffers from the MES4-CIF §2c table: no relay coil feedback, so PA0-PA3 drive the winch and the servo UART.\nRelay drive per CIF §7a (AO3400A, 100 Ω, 100k pull-down); the Flasher uses a 2SC2884 BJT for the same job.\nNo hot-plug: unplug the 24 V XT30 before inserting or removing the module.\nPages: Main (2), CAN (3), Power (4), Relays 1-2 (5), Relays 3-4 (6), Sensors (7), LoadCell (8), AuxPower (9), Winch (10)."
 		(exclude_from_sim no)
 		(at 20.32 221 0)
@@
 		(instances
 			(project "MES4_Carrier_EC"
-				(path "/86b406aa-a59b-5773-8968-b904bb1c5afe"
+				(path "/20e873b0-a362-5816-a506-9e1cffc294d3"
 					(page "2")
 				)
@@
 		(instances
 			(project "MES4_Carrier_EC"
-				(path "/86b406aa-a59b-5773-8968-b904bb1c5afe"
+				(path "/20e873b0-a362-5816-a506-9e1cffc294d3"
 					(page "3")
 				)
@@
 		(instances
 			(project "MES4_Carrier_EC"
-				(path "/86b406aa-a59b-5773-8968-b904bb1c5afe"
+				(path "/20e873b0-a362-5816-a506-9e1cffc294d3"
 					(page "4")
 				)
@@
 		(instances
 			(project "MES4_Carrier_EC"
-				(path "/86b406aa-a59b-5773-8968-b904bb1c5afe"
+				(path "/20e873b0-a362-5816-a506-9e1cffc294d3"
 					(page "5")
 				)
@@
 		(instances
 			(project "MES4_Carrier_EC"
-				(path "/86b406aa-a59b-5773-8968-b904bb1c5afe"
+				(path "/20e873b0-a362-5816-a506-9e1cffc294d3"
 					(page "6")
 				)
@@
 		(instances
 			(project "MES4_Carrier_EC"
-				(path "/86b406aa-a59b-5773-8968-b904bb1c5afe"
+				(path "/20e873b0-a362-5816-a506-9e1cffc294d3"
 					(page "7")
 				)
@@
 		(instances
 			(project "MES4_Carrier_EC"
-				(path "/86b406aa-a59b-5773-8968-b904bb1c5afe"
+				(path "/20e873b0-a362-5816-a506-9e1cffc294d3"
 					(page "8")
 				)
@@
 		(instances
 			(project "MES4_Carrier_EC"
-				(path "/86b406aa-a59b-5773-8968-b904bb1c5afe"
+				(path "/20e873b0-a362-5816-a506-9e1cffc294d3"
 					(page "9")
 				)
@@
 		(instances
 			(project "MES4_Carrier_EC"
-				(path "/86b406aa-a59b-5773-8968-b904bb1c5afe"
+				(path "/20e873b0-a362-5816-a506-9e1cffc294d3"
 					(page "10")
 				)
