File: MES4_Carrier_EC/MES4_Carrier_EC.kicad_sch (KiCad schematic)
At the start: 0 parts

Commit message: Address design review R1: INA236, J15 polarity, review fixes
M1: U2-U5 are now TI INA236AIDDFR (C5443912, 50 V abs max, TSOT-23-8)
instead of the INA226 (40 V), since the SMBJ30A clamps at up to 48.4 V.
A project INA236 symbol keeps the INA226 body so the Flasher relay
wiring lands on the same pins; A1 and VBUS are gone (bus read on IN-),
addresses 0x40-0x43 via A0 = GND / VS / SDA / SCL. Same CONFIG / CAL /
MASK / ALERT values; notes give the 1.6 mV bus LSB and Device ID.
M3: J15 servo 24 V is pin 1 = +24 V like every power terminal.
L4: R38 servo RX series resistor 1k (limits PA3 back-feed).
L2: "current present" threshold 3 mA. L6: Power notes use 13 A / 2.2 W.
M2 / L5: silkscreen notes for "5V LOAD CELL - NEVER 24V" and
"CAN - NOT ETHERNET" (no keyed connector, by choice).
RJ45 1x4 footprint rebuilt from the HCTL drawing (14.0 mm ports,
Ø1.5 shield and Ø3.2 peg positions); U1 / U9 / U10 checked against the
JLC library and YLPTEC drawing. HANDOFF gains the review status table
and a layout checklist.

Co-Authored-By: Claude Opus 5.5 <noreply@anthropic.com>
Other:
- note added: "+24V rail: relay contacts, INA236 monitors, sensor supplies, servo and aux power"
- note added: "1 safety light: PA8 drive, INA236 0x40 2 LED DRL: PC6 drive, INA236 0x41 3 battery stopper: PB3 drive, INA236 0x42 4 spare: PA7 drive, INA236 0x43 GPIO → 100 Ω → AO3400A → 5 V coil (SRD-5VDC-SL-A, on +5V_24). +24V → 30 mΩ shunt → contact → 3A PTC → output (2 A continuous). No coil feedback (pins used elsewhere). INA236 per channel: load current + 24 V rail, ALERT → PA15."
- note added: "E-Crawler carrier for one MES4-MCU module (MES4-CIF rev A-d6). Circuits taken from the MES4-Flasher: PC817 sensor inputs, ADS1232 load cell, relay channels (driver, current monitor) and the XT30 / URB2405S 24 V input. GPIO budget: 4 relay drives + ALERT + 3 ADS1232 + 2 sensors + winch (2) + servo USART2 (2) = 14. Differs from the MES4-CIF §2c table: no relay coil feedback, so PA0-PA3 drive the wi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"
- note added: "J15: +24V → F9 3 A PTC → FE-URT-2 → Feetech servos (24 V types). J17: USART2 PA2 TX / PA3 RX (100 Ω / 1k) + ESD. FE-URT-2 set to 3.3 V levels; its 5 V logic supply comes from the screen converter."
- note added: "STM32G0B1, 64 MHz, CAN transceiver. Gets +5V on fingers 20 / 22. Makes its own 3.3 V → +3V3_MOD (finger 4, ≤ 50 mA) for the I²C pull-ups, INA236s, PC817 outputs and the ADS1232 logic. All 14 GPIOs are used (GPIO map on the Main sheet). LED1 = module +5V, LED2 = 3V3. Hold-down: H1 M3 standoff. No hot-plug: unplug the XT30 before fitting a module."
- note removed: "+24V rail: relay contacts, INA226 VBUS, sensor supplies, servo and aux power"
- note removed: "1 safety light: PA8 drive, INA226 0x40 2 LED DRL: PC6 drive, INA226 0x41 3 battery stopper: PB3 drive, INA226 0x44 4 spare: PA7 drive, INA226 0x45 GPIO → 100 Ω → AO3400A → 5 V coil (SRD-5VDC-SL-A, on +5V_24). +24V → 30 mΩ shunt → contact → 3A PTC → output (2 A continuous). No coil feedback (pins used elsewhere). INA226 per channel: load current + 24 V rail, ALERT → PA15."
- note removed: "E-Crawler carrier for one MES4-MCU module (MES4-CIF rev A-d6). Circuits taken from the MES4-Flasher: PC817 sensor inputs, ADS1232 load cell, relay channels (driver, INA226) and the XT30 / URB2405S 24 V input. GPIO budget: 4 relay drives + ALERT + 3 ADS1232 + 2 sensors + winch (2) + servo USART2 (2) = 14. Differs from the MES4-CIF §2c table: no relay coil feedback, so PA0-PA3 drive the winch and t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"
- note removed: "J15: +24V → F9 3 A PTC → FE-URT-2 → Feetech servos (24 V types). J17: USART2 PA2 TX / PA3 RX, 100 Ω + ESD. FE-URT-2 set to 3.3 V levels; its 5 V logic supply comes from the screen converter."
- note removed: "STM32G0B1, 64 MHz, CAN transceiver. Gets +5V on fingers 20 / 22. Makes its own 3.3 V → +3V3_MOD (finger 4, ≤ 50 mA) for the I²C pull-ups, INA226s, PC817 outputs and the ADS1232 logic. All 14 GPIOs are used (GPIO map on the Main sheet). LED1 = module +5V, LED2 = 3V3. Hold-down: H1 M3 standoff. No hot-plug: unplug the XT30 before fitting a module."
Changed lines of the file:
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@@
 		(effects (font (size 2.2 2.2) (bold yes)) (justify left top))
 	)
-	(text "STM32G0B1, 64 MHz, CAN transceiver.\nGets +5V on fingers 20 / 22.\nMakes its own 3.3 V → +3V3_MOD\n(finger 4, ≤ 50 mA) for the I²C\npull-ups, INA226s, PC817 outputs\nand the ADS1232 logic.\n\nAll 14 GPIOs are used\n(GPIO map on the Main sheet).\n\nLED1 = module +5V, LED2 = 3V3.\nHold-down: H1 M3 standoff.\n\nNo hot-plug: unplug the XT30\nbefore fitting a module."
+	(text "STM32G0B1, 64 MHz, CAN transceiver.\nGets +5V on fingers 20 / 22.\nMakes its own 3.3 V → +3V3_MOD\n(finger 4, ≤ 50 mA) for the I²C\npull-ups, INA236s, PC817 outputs\nand the ADS1232 logic.\n\nAll 14 GPIOs are used\n(GPIO map on the Main sheet).\n\nLED1 = module +5V, LED2 = 3V3.\nHold-down: H1 M3 standoff.\n\nNo hot-plug: unplug the XT30\nbefore fitting a module."
 		(exclude_from_sim no)
 		(at 109.22 48.26 0)
@@
 		(effects (font (size 2.2 2.2) (bold yes)) (justify left top))
 	)
-	(text "1 safety light: PA8 drive, INA226 0x40\n2 LED DRL: PC6 drive, INA226 0x41\n3 battery stopper: PB3 drive, INA226 0x44\n4 spare: PA7 drive, INA226 0x45\n\nGPIO → 100 Ω → AO3400A → 5 V coil\n(SRD-5VDC-SL-A, on +5V_24).\n+24V → 30 mΩ shunt → contact →\n3A PTC → output (2 A continuous).\nNo coil feedback (pins used elsewhere).\nINA226 per channel: load current +\n24 V rail, ALERT → PA15."
+	(text "1 safety light: PA8 drive, INA236 0x40\n2 LED DRL: PC6 drive, INA236 0x41\n3 battery stopper: PB3 drive, INA236 0x42\n4 spare: PA7 drive, INA236 0x43\n\nGPIO → 100 Ω → AO3400A → 5 V coil\n(SRD-5VDC-SL-A, on +5V_24).\n+24V → 30 mΩ shunt → contact →\n3A PTC → output (2 A continuous).\nNo coil feedback (pins used elsewhere).\nINA236 per channel: load current +\n24 V rail, ALERT → PA15."
 		(exclude_from_sim no)
 		(at 208.28 48.26 0)
@@
 		(fill (type color) (color 200 30 30 1))
 	)
-	(text "+24V rail: relay contacts, INA226 VBUS, sensor supplies, servo and aux power"
+	(text "+24V rail: relay contacts, INA236 monitors, sensor supplies, servo and aux power"
 		(exclude_from_sim no)
 		(at 120.65 29.21 0)
@@
 		(effects (font (size 2.2 2.2) (bold yes)) (justify left top))
 	)
-	(text "J15: +24V → F9 3 A PTC → FE-URT-2\n→ Feetech servos (24 V types).\nJ17: USART2 PA2 TX / PA3 RX, 100 Ω + ESD.\nFE-URT-2 set to 3.3 V levels; its 5 V\nlogic supply comes from the screen converter."
+	(text "J15: +24V → F9 3 A PTC → FE-URT-2\n→ Feetech servos (24 V types).\nJ17: USART2 PA2 TX / PA3 RX (100 Ω / 1k) + ESD.\nFE-URT-2 set to 3.3 V levels; its 5 V\nlogic supply comes from the screen converter."
 		(exclude_from_sim no)
 		(at 320.04 83.82 0)
@@
 		(effects (font (size 2.2 2.2) (bold yes)) (justify left top))
 	)
-	(text "E-Crawler carrier for one MES4-MCU module (MES4-CIF rev A-d6). Circuits taken from the MES4-Flasher: PC817 sensor inputs,\nADS1232 load cell, relay channels (driver, INA226) and the XT30 / URB2405S 24 V input.\nGPIO budget: 4 relay drives + ALERT + 3 ADS1232 + 2 sensors + winch (2) + servo USART2 (2) = 14.\nDiffers from the MES4-CIF §2c table: no relay coil feedback, so PA0-PA3 drive the winch and the servo UART.\nRelay drive per CIF §7a (AO3400A, 100 Ω, 100k pull-down); the Flasher uses a 2SC2884 BJT for the same job.\nNo hot-plug: unplug the 24 V XT30 before inserting or removing the module.\nPages: Main (2), CAN (3), Power (4), Relays 1-2 (5), Relays 3-4 (6), Sensors (7), LoadCell (8), AuxPower (9), Winch (10), Pinout (11)."
+	(text "E-Crawler carrier for one MES4-MCU module (MES4-CIF rev A-d6). Circuits taken from the MES4-Flasher: PC817 sensor inputs,\nADS1232 load cell, relay channels (driver, current monitor) and the XT30 / URB2405S 24 V input.\nGPIO budget: 4 relay drives + ALERT + 3 ADS1232 + 2 sensors + winch (2) + servo USART2 (2) = 14.\nDiffers from the MES4-CIF §2c table: no relay coil feedback, so PA0-PA3 drive the winch and the servo UART.\nRelay drive per CIF §7a (AO3400A, 100 Ω, 100k pull-down); the Flasher uses a 2SC2884 BJT for the same job.\nNo hot-plug: unplug the 24 V XT30 before inserting or removing the module.\nPages: Main (2), CAN (3), Power (4), Relays 1-2 (5), Relays 3-4 (6), Sensors (7), LoadCell (8), AuxPower (9), Winch (10), Pinout (11)."
 		(exclude_from_sim no)
 		(at 20.32 221 0)
@@
 		(instances
 			(project "MES4_Carrier_EC"
-				(path "/0370b922-a365-5c71-ab6f-f5cfbc7b5e5a"
+				(path "/0d8fbf0e-dd62-5be6-8889-307c6423adb0"
 					(page "2")
 				)
@@
 		(instances
 			(project "MES4_Carrier_EC"
-				(path "/0370b922-a365-5c71-ab6f-f5cfbc7b5e5a"
+				(path "/0d8fbf0e-dd62-5be6-8889-307c6423adb0"
 					(page "3")
 				)
@@
 		(instances
 			(project "MES4_Carrier_EC"
-				(path "/0370b922-a365-5c71-ab6f-f5cfbc7b5e5a"
+				(path "/0d8fbf0e-dd62-5be6-8889-307c6423adb0"
 					(page "4")
 				)
@@
 		(instances
 			(project "MES4_Carrier_EC"
-				(path "/0370b922-a365-5c71-ab6f-f5cfbc7b5e5a"
+				(path "/0d8fbf0e-dd62-5be6-8889-307c6423adb0"
 					(page "5")
 				)
@@
 		(instances
 			(project "MES4_Carrier_EC"
-				(path "/0370b922-a365-5c71-ab6f-f5cfbc7b5e5a"
+				(path "/0d8fbf0e-dd62-5be6-8889-307c6423adb0"
 					(page "6")
 				)
@@
 		(instances
 			(project "MES4_Carrier_EC"
-				(path "/0370b922-a365-5c71-ab6f-f5cfbc7b5e5a"
+				(path "/0d8fbf0e-dd62-5be6-8889-307c6423adb0"
 					(page "7")
 				)
@@
 		(instances
 			(project "MES4_Carrier_EC"
-				(path "/0370b922-a365-5c71-ab6f-f5cfbc7b5e5a"
+				(path "/0d8fbf0e-dd62-5be6-8889-307c6423adb0"
 					(page "8")
 				)
@@
 		(instances
 			(project "MES4_Carrier_EC"
-				(path "/0370b922-a365-5c71-ab6f-f5cfbc7b5e5a"
+				(path "/0d8fbf0e-dd62-5be6-8889-307c6423adb0"
 					(page "9")
 				)
@@
 		(instances
 			(project "MES4_Carrier_EC"
-				(path "/0370b922-a365-5c71-ab6f-f5cfbc7b5e5a"
+				(path "/0d8fbf0e-dd62-5be6-8889-307c6423adb0"
 					(page "10")
 				)
@@
 		(instances
 			(project "MES4_Carrier_EC"
-				(path "/0370b922-a365-5c71-ab6f-f5cfbc7b5e5a"
+				(path "/0d8fbf0e-dd62-5be6-8889-307c6423adb0"
 					(page "11")
 				)

Commit message: PCB placement, FE-URT-2 and GPS mounts, smaller screen converter, review R3
Placement: all terminals, USB-C and XT30 face the top edge (CAN DB9/RJ45 on
the sides), power block (U1, U9, U10, filters, GND joint) under the 24 V
input, relay bank and winch block below the terminal row, MES4-MCU slot
grouped with the Flasher's slot silkscreen. Feetech and GPS mounts parked
off-board until the layout is final.

Mounts: FE-URT-2 on 4 x YIYUAN SMTSOM320BTR M3 x 2 mm SMD standoffs (H6-H9,
C5301780) as on the MES3 carriers, board-only outline with a footprint
keep-out; simpleRTK4 Dual on 3 x SMTSOM365BTR M3 x 6.5 mm standoffs
(H10-H12, C5301796) + 12 mm spacers, with its STEP.

U10: URB2405LD-20WR3 (2" x 1") -> YLPTEC URB2405YMD-20WR3 (1" x 1",
C5369777), footprint from the JLC part checked against the Mornsun drawing;
C38 100 uF / 16 V output bulk (C81993) per its datasheet. AUX1 re-run:
3.58 A start-up peak vs 4.4 A OCP, 3.0 A at 4.94 V. Review package R3.

Generator: new parts take UUIDs from their own counter range so no PCB link
moves; import_footprints.py --add-missing; group_footprints.py never moves
placed parts and stops once groups are edited in KiCad.

Co-Authored-By: Claude Opus 5.5 <noreply@anthropic.com>
Other:
- note added: "Own L pi filter from +24V. U9 URB2409S-10WR3 → 9 V → SW2 switch → J14 IMU terminal (as on the MES3.1 carrier). U10 URB2405YMD-20WR3 → 5 V 4 A → 3 A PTC → J16 USB-C (Rp 10k: 5 V / 3 A) → ARZOPA Z1C screen."
- note removed: "Own L pi filter from +24V. U9 URB2409S-10WR3 → 9 V → SW2 switch → J14 IMU terminal (as on the MES3.1 carrier). U10 URB2405LD-20WR3 → 5 V 4 A → 3 A PTC → J16 USB-C (Rp 10k: 5 V / 3 A) → ARZOPA Z1C screen."
Changed lines of the file:
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@@
 		(effects (font (size 2.2 2.2) (bold yes)) (justify left top))
 	)
-	(text "Own L pi filter from +24V.\nU9 URB2409S-10WR3 → 9 V →\nSW2 switch → J14 IMU terminal\n(as on the MES3.1 carrier).\nU10 URB2405LD-20WR3 → 5 V 4 A\n→ 3 A PTC → J16 USB-C (Rp 10k:\n5 V / 3 A) → ARZOPA Z1C screen."
+	(text "Own L pi filter from +24V.\nU9 URB2409S-10WR3 → 9 V →\nSW2 switch → J14 IMU terminal\n(as on the MES3.1 carrier).\nU10 URB2405YMD-20WR3 → 5 V 4 A\n→ 3 A PTC → J16 USB-C (Rp 10k:\n5 V / 3 A) → ARZOPA Z1C screen."
 		(exclude_from_sim no)
 		(at 320.04 119.38 0)

Commit message: Fix design review R3 findings: U9 part, stale LCSC fields, labels, J16
- B1: U9 is now YLPTEC URB2409S-6WR3 (C7468814, 9 V 6 W) on U1's
  footprint; the 10 W URB2409S-10WR3 isn't in JLC's assembly library.
  The production BOM had a 5 V module at U9 and the wrong SW2 because
  EasyEDA footprints carry an "LCSC Part" field the Fabrication Toolkit
  reads first: libs.py strips it (and the unprintable pin-1 dots it was
  copying back), and the new parts_sync.py syncs board footprints,
  values, fields and BOM flags from the schematic. TP1-TP9 and H2-H5
  are out of the BOM and CPL.
- M2 / L5: "5V LOAD CELL" across J12 / J13; "CANBUS" knockout by J4.
- B2: J16 moves 1.25 mm west so its mouth reaches the board edge.
- B8 / N6: README (one ground, U9, J16, labels, TPs), schematic notes
  and HANDOFF updated; 1:1 A4 print refreshed.
- DRC with parity at the 3 accepted J4 notes; nets, audit, DFM clean.
  production/ is stale until the Fabrication Toolkit is re-run.

Co-Authored-By: Claude Opus 5.5 <noreply@anthropic.com>
Other:
- note added: "Own L pi filter from +24V. U9 URB2409S-6WR3 → 9 V → SW2 switch → J14 IMU terminal (as on the MES3.1 carrier). U10 URB2405YMD-20WR3 → 5 V 4 A → 3 A PTC → J16 USB-C (Rp 10k: 5 V / 3 A) → ARZOPA Z1C screen."
- note removed: "Own L pi filter from +24V. U9 URB2409S-10WR3 → 9 V → SW2 switch → J14 IMU terminal (as on the MES3.1 carrier). U10 URB2405YMD-20WR3 → 5 V 4 A → 3 A PTC → J16 USB-C (Rp 10k: 5 V / 3 A) → ARZOPA Z1C screen."
Changed lines of the file:
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@@
 		(effects (font (size 2.2 2.2) (bold yes)) (justify left top))
 	)
-	(text "Own L pi filter from +24V.\nU9 URB2409S-10WR3 → 9 V →\nSW2 switch → J14 IMU terminal\n(as on the MES3.1 carrier).\nU10 URB2405YMD-20WR3 → 5 V 4 A\n→ 3 A PTC → J16 USB-C (Rp 10k:\n5 V / 3 A) → ARZOPA Z1C screen."
+	(text "Own L pi filter from +24V.\nU9 URB2409S-6WR3 → 9 V →\nSW2 switch → J14 IMU terminal\n(as on the MES3.1 carrier).\nU10 URB2405YMD-20WR3 → 5 V 4 A\n→ 3 A PTC → J16 USB-C (Rp 10k:\n5 V / 3 A) → ARZOPA Z1C screen."
 		(exclude_from_sim no)
 		(at 320.04 119.38 0)
