File: MES4_Carrier_EC/Main.kicad_sch (KiCad schematic)
At the start: 20 parts, among them J1 2199230-3, J2 STDC14, SW1 RESET

Commit message: Address design review R1: INA236, J15 polarity, review fixes
M1: U2-U5 are now TI INA236AIDDFR (C5443912, 50 V abs max, TSOT-23-8)
instead of the INA226 (40 V), since the SMBJ30A clamps at up to 48.4 V.
A project INA236 symbol keeps the INA226 body so the Flasher relay
wiring lands on the same pins; A1 and VBUS are gone (bus read on IN-),
addresses 0x40-0x43 via A0 = GND / VS / SDA / SCL. Same CONFIG / CAL /
MASK / ALERT values; notes give the 1.6 mV bus LSB and Device ID.
M3: J15 servo 24 V is pin 1 = +24 V like every power terminal.
L4: R38 servo RX series resistor 1k (limits PA3 back-feed).
L2: "current present" threshold 3 mA. L6: Power notes use 13 A / 2.2 W.
M2 / L5: silkscreen notes for "5V LOAD CELL - NEVER 24V" and
"CAN - NOT ETHERNET" (no keyed connector, by choice).
RJ45 1x4 footprint rebuilt from the HCTL drawing (14.0 mm ports,
Ø1.5 shield and Ø3.2 peg positions); U1 / U9 / U10 checked against the
JLC library and YLPTEC drawing. HANDOFF gains the review status table
and a layout checklist.

Co-Authored-By: Claude Opus 5.5 <noreply@anthropic.com>
Other:
- note added: "CIF rule 7: always fitted, to the module's 3V3 (finger 4). 2.2k: 4 × INA236 at 400 kHz. R5: INA236 ALERT wire-OR (PA15)."
- note added: "Module CANH / CANL (fingers 1 / 3) go to the CAN sheet as global labels: J3 DB9 male to the IPC: 1 GND, 3 CAN_H, 5 CAN_L. J4 1x4 RJ45, no magnetics: 1 CAN_H, 2 CAN_L, 3 GND on every port (T568B: white-orange, orange, white-green). All five ports are one bus, wired in parallel. ESD at each connector: D6, D7 (H24VNT2B). Transceiver + 120 Ω terminator (JP1) are on the module. Silkscreen + panel at J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"
- note added: "Page 1: block diagram and page list. Page 3 CAN: DB9 male to the IPC + 1x4 RJ45, ESD. Page 4 Power: XT30 24 V input, fuse, reverse-polarity FET, TVS, noise filter, 24 V → 5 V. Pages 5-6 Relays: PA8 / PC6 / PB3 / PA7 drive, 4 × INA236 (no coil feedback). Page 7 Sensors: PB6 / PC15 (two Autonics PNP sensors). Page 8 LoadCell: PA4 DRDY, PA5 SCLK, PA6 PDWN. Page 9 AuxPower: IMU 9 V (MES3.1), screen U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"
- note removed: "CIF rule 7: always fitted, to the module's 3V3 (finger 4). 2.2k: 4 × INA226 at 400 kHz. R5: INA226 ALERT wire-OR (PA15)."
- note removed: "Module CANH / CANL (fingers 1 / 3) go to the CAN sheet as global labels: J3 DB9 male to the IPC: 1 GND, 3 CAN_H, 5 CAN_L. J4 1x4 RJ45, no magnetics: 1 CAN_H, 2 CAN_L, 3 GND on every port (T568B: white-orange, orange, white-green). All five ports are one bus, wired in parallel. ESD at each connector: D6, D7 (H24VNT2B). Transceiver + 120 Ω terminator (JP1) are on the module."
- note removed: "Page 1: block diagram and page list. Page 3 CAN: DB9 male to the IPC + 1x4 RJ45, ESD. Page 4 Power: XT30 24 V input, fuse, reverse-polarity FET, TVS, noise filter, 24 V → 5 V. Pages 5-6 Relays: PA8 / PC6 / PB3 / PA7 drive, 4 × INA226 (no coil feedback). Page 7 Sensors: PB6 / PC15 (two Autonics PNP sensors). Page 8 LoadCell: PA4 DRDY, PA5 SCLK, PA6 PDWN. Page 9 AuxPower: IMU 9 V (MES3.1), screen U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"

Commit message: Add whole-board LTspice simulations, IMU notes and the R2 review package
sim/: 16 LTspice benches grouped by schematic sheet (Power, Relays,
Sensors, LoadCell, AuxPower, IMU, Winch, Main) on the real supply chain
(DDR-480C-24 at 24 V and a 24 V Li-ion pack via XY-CD63L, diode-OR'd by
an Autoro AB20). run_sims.py runs them, make_report.py builds
report.html. All pass; the IEC 0.5 kV surge is not applicable to this
internal, isolated supply. Raw waveforms and logs are git-ignored.

IMU: 3DM-CV7-AHRS on the C-Series Connectivity Board (6212-3009). The
AuxPower and Main notes, README and HANDOFF now say J14's 9 V goes to the
board's Vaux only (never Vpri), not together with the USB cable; the
power budget uses the real ~0.02 A at 24 V.

review/: MES4-Carrier-EC_Review-Package_R2.pdf, 26 pages: changes since
R1, status of every R1 finding, open items, the simulation report and
the regenerated 11-page schematic. HANDOFF records the supply chain and
the M4 results.

Co-Authored-By: Claude Opus 5.5 <noreply@anthropic.com>
Changed lines of the file:
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@@
 		(effects (font (size 2 2) (bold yes)) (justify left top))
 	)
-	(text "J5 24V IN, XT30 male right-angle: 1 = +24 V (flat end),\n   2 = GND_24V (chamfered end).\nJ6 / J7 / J8 / J9 RLY1-4 OUT (KF250NH 2-pin):\n   1 = switched +24 V, 2 = GND_24V.\nJ10 / J11 SENS1 / SENS2 (KF250NH 3-pin): 1 = +24 V\n   (100 mA PTC, brown), 2 = output (black), 3 = 0 V (blue).\nJ12 LC SIG: 1 SIG+ green, 2 SIG- white, 3 shield.\nJ13 LC EXC: 1 EXC+ red, 2 EXC- black, 3 shield.\n   5 V load cell only: never 24 V.\nJ3 CAN DB9 male (IPC): 1 GND, 3 CAN_H, 5 CAN_L.\nJ4 CAN RJ45 x4: 1 CAN_H, 2 CAN_L, 3 GND (T568B).\nJ14 IMU 9V (KF250NH 2-pin): 1 = +9 V after the switch, 2 = GND.\nJ16 SCREEN USB-C: 5 V / 3 A power only (no data).\nJ15 SERVO 24V: 1 +24 V (3 A PTC), 2 GND_24V.\nJ17 SERVO UART: 1 GND, 2 +5 V, 3 RX, 4 TX.\nJ18 WINCH: 1 CLK, 2 COM, 3 ACLK (relay contacts).\nJ2 STDC14: ST-Link V3MINIE (SWD, NRST, VCP).\nTest points: Power sheet."
+	(text "J5 24V IN, XT30 male right-angle: 1 = +24 V (flat end),\n   2 = GND_24V (chamfered end).\nJ6 / J7 / J8 / J9 RLY1-4 OUT (KF250NH 2-pin):\n   1 = switched +24 V, 2 = GND_24V.\nJ10 / J11 SENS1 / SENS2 (KF250NH 3-pin): 1 = +24 V\n   (100 mA PTC, brown), 2 = output (black), 3 = 0 V (blue).\nJ12 LC SIG: 1 SIG+ green, 2 SIG- white, 3 shield.\nJ13 LC EXC: 1 EXC+ red, 2 EXC- black, 3 shield.\n   5 V load cell only: never 24 V.\nJ3 CAN DB9 male (IPC): 1 GND, 3 CAN_H, 5 CAN_L.\nJ4 CAN RJ45 x4: 1 CAN_H, 2 CAN_L, 3 GND (T568B).\nJ14 IMU 9V (KF250NH 2-pin): 1 = +9 V after the switch, 2 = GND. To the CV7 dev board Vaux only.\nJ16 SCREEN USB-C: 5 V / 3 A power only (no data).\nJ15 SERVO 24V: 1 +24 V (3 A PTC), 2 GND_24V.\nJ17 SERVO UART: 1 GND, 2 +5 V, 3 RX, 4 TX.\nJ18 WINCH: 1 CLK, 2 COM, 3 ACLK (relay contacts).\nJ2 STDC14: ST-Link V3MINIE (SWD, NRST, VCP).\nTest points: Power sheet."
 		(exclude_from_sim no)
 		(at 165.1 191.77 0)

Commit message: One ground and a 4-layer board
- GND_24V merged into GND (ONE_GND in gen.py): every GND_24V power symbol
  becomes GND, net tie NT1 left out, notes reworded. Symbol UUIDs unchanged,
  so every footprint keeps its link.
- 4 layers, JLC04161H-7628 stackup (1.6 mm, ENIG): Top Signal / GND plane
  (In1) / +24V plane (In2) / Bottom Signal.
- Net classes: Out_3A (1.5 mm) for +24V_SRV, +5V_SCR, VBUS_SCR; +24V_AUX to
  24V_Power; +5V_SRV, +9V_IMU, IMU_9V to Power; INA236 shunt pattern fixed
  (Net-(U*-IN-)).
- J1's NPTH holes back to F&B.Cu as in its library footprint.

ERC 0, checks passed, DRC 11 silkscreen warnings, schematic parity clean.

Co-Authored-By: Claude Opus 5.5 <noreply@anthropic.com>
Other:
- note added: "J5 24V IN, XT30 male right-angle: 1 = +24 V (flat end), 2 = GND (chamfered end). J6 / J7 / J8 / J9 RLY1-4 OUT (KF250NH 2-pin): 1 = switched +24 V, 2 = GND. J10 / J11 SENS1 / SENS2 (KF250NH 3-pin): 1 = +24 V (100 mA PTC, brown), 2 = output (black), 3 = 0 V (blue). J12 LC SIG: 1 SIG+ green, 2 SIG- white, 3 shield. J13 LC EXC: 1 EXC+ red, 2 EXC- black, 3 shield. 5 V load cell only: never 24 V. J3 CA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"
- note removed: "J5 24V IN, XT30 male right-angle: 1 = +24 V (flat end), 2 = GND_24V (chamfered end). J6 / J7 / J8 / J9 RLY1-4 OUT (KF250NH 2-pin): 1 = switched +24 V, 2 = GND_24V. J10 / J11 SENS1 / SENS2 (KF250NH 3-pin): 1 = +24 V (100 mA PTC, brown), 2 = output (black), 3 = 0 V (blue). J12 LC SIG: 1 SIG+ green, 2 SIG- white, 3 shield. J13 LC EXC: 1 EXC+ red, 2 EXC- black, 3 shield. 5 V load cell only: never 24 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"

Commit message: Fix design review R3 findings: U9 part, stale LCSC fields, labels, J16
- B1: U9 is now YLPTEC URB2409S-6WR3 (C7468814, 9 V 6 W) on U1's
  footprint; the 10 W URB2409S-10WR3 isn't in JLC's assembly library.
  The production BOM had a 5 V module at U9 and the wrong SW2 because
  EasyEDA footprints carry an "LCSC Part" field the Fabrication Toolkit
  reads first: libs.py strips it (and the unprintable pin-1 dots it was
  copying back), and the new parts_sync.py syncs board footprints,
  values, fields and BOM flags from the schematic. TP1-TP9 and H2-H5
  are out of the BOM and CPL.
- M2 / L5: "5V LOAD CELL" across J12 / J13; "CANBUS" knockout by J4.
- B2: J16 moves 1.25 mm west so its mouth reaches the board edge.
- B8 / N6: README (one ground, U9, J16, labels, TPs), schematic notes
  and HANDOFF updated; 1:1 A4 print refreshed.
- DRC with parity at the 3 accepted J4 notes; nets, audit, DFM clean.
  production/ is stale until the Fabrication Toolkit is re-run.

Co-Authored-By: Claude Opus 5.5 <noreply@anthropic.com>
Other:
- note added: "Module CANH / CANL (fingers 1 / 3) go to the CAN sheet as global labels: J3 DB9 male to the IPC: 1 GND, 3 CAN_H, 5 CAN_L. J4 1x4 RJ45, no magnetics: 1 CAN_H, 2 CAN_L, 3 GND on every port (T568B: white-orange, orange, white-green). All five ports are one bus, wired in parallel. ESD at each connector: D6, D7 (H24VNT2B). Transceiver + 120 Ω terminator (JP1) are on the module. Silkscreen at J4: a "CA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"
- note removed: "Module CANH / CANL (fingers 1 / 3) go to the CAN sheet as global labels: J3 DB9 male to the IPC: 1 GND, 3 CAN_H, 5 CAN_L. J4 1x4 RJ45, no magnetics: 1 CAN_H, 2 CAN_L, 3 GND on every port (T568B: white-orange, orange, white-green). All five ports are one bus, wired in parallel. ESD at each connector: D6, D7 (H24VNT2B). Transceiver + 120 Ω terminator (JP1) are on the module. Silkscreen + panel at J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"
Changed lines of the file:
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@@
 		(effects (font (size 2 2) (bold yes)) (justify left top))
 	)
-	(text "Module CANH / CANL (fingers 1 / 3) go to the CAN sheet\nas global labels:\n\nJ3 DB9 male to the IPC: 1 GND, 3 CAN_H, 5 CAN_L.\nJ4 1x4 RJ45, no magnetics: 1 CAN_H, 2 CAN_L,\n3 GND on every port (T568B: white-orange, orange,\nwhite-green).\n\nAll five ports are one bus, wired in parallel.\nESD at each connector: D6, D7 (H24VNT2B).\nTransceiver + 120 Ω terminator (JP1) are on the module.\nSilkscreen + panel at J4: \"CAN - NOT ETHERNET\" (review L5)."
+	(text "Module CANH / CANL (fingers 1 / 3) go to the CAN sheet\nas global labels:\n\nJ3 DB9 male to the IPC: 1 GND, 3 CAN_H, 5 CAN_L.\nJ4 1x4 RJ45, no magnetics: 1 CAN_H, 2 CAN_L,\n3 GND on every port (T568B: white-orange, orange,\nwhite-green).\n\nAll five ports are one bus, wired in parallel.\nESD at each connector: D6, D7 (H24VNT2B).\nTransceiver + 120 Ω terminator (JP1) are on the module.\nSilkscreen at J4: a \"CANBUS\" knockout; mark the panel\nthe same, so nobody plugs Ethernet in (review L5)."
 		(exclude_from_sim no)
 		(at 317.5 30.48 0)
