File: MES4_Carrier_EC/Relays12.kicad_sch (KiCad schematic)
At the start: 26 parts, among them J6 RLY1 OUT, J7 RLY2 OUT, K1 SRD-5VDC-SL-A, K2 SRD-5VDC-SL-A, Q2 AO3400A, Q3 AO3400A, U2 INA236, U3 INA236

Commit message: Check CPL rotations against JLC's footprints; fix Q1, K1-K4, J5
- cpl_check.py: fetches each LCSC part's EasyEDA footprint, matches
  pads (polarity names, numbers or shape), fits the rotation / offset
  JLC needs and compares with production/positions.csv.
- Q1 (TO-252) needs +180 deg and -1.8 mm, K1-K4 (SRD relays) +180 deg,
  J5 (XT30) +9.7 mm: set as Fabrication Toolkit FT Rotation / Position
  Offset fields on the symbols (gen.py, parts.py), copied to the board
  by parts_sync.py.
- production/ regenerated with the toolkit CLI: 169 of 181 placements
  match JLC; C1 / C5 / C27 (no JLC footprint) to check in the preview.
- HANDOFF updated.

Co-Authored-By: Claude Opus 5.5 <noreply@anthropic.com>
Parts:
- K1, K2: FT Rotation Offset (none) -> 180
Changed lines of the file:
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@@
+			(effects (font (size 1.27 1.27)) (hide yes))
+		)
+		(property "FT Rotation Offset" "180"
+			(at 172.72 66.04 0)
 			(effects (font (size 1.27 1.27)) (hide yes))
 		)
@@
 			(at 172.72 170.18 0)
 			(effects (font (size 1.27 1.27)) (hide yes))
+		)
+		(property "FT Rotation Offset" "180"
+			(at 172.72 170.18 0)
+			(effects (font (size 1.27 1.27)) (hide yes))
