File: MES4_Carrier_EC/Relays12.kicad_sch (KiCad schematic)
At the start: 26 parts, among them J6 RLY1 OUT, J7 RLY2 OUT, K1 SRD-5VDC-SL-A, K2 SRD-5VDC-SL-A, Q2 AO3400A, Q3 AO3400A, U2 INA236, U3 INA236

Commit message: Fix design review R4 (CPL), add 3D models, STEP and the enclosure
Review R4:
- E1 (blocking): the Fabrication Toolkit turns every CP_Elec 180 deg, but
  JLC's footprints for C1/C5/C27/C28/C30/C32/C38 have + on the same side
  as ours, so all seven would have been fitted reversed. gen.py now sets
  FT Rotation Offset 180 on every CP_Elec part (the toolkit adds it to its
  own 180), so the CPL keeps the board rotation.
- E2: J5's FT Position Offset 0,9.7 put the XT30 10 mm off; JLC's origin
  is ours. Removed; parts_sync.py now drops FT fields the schematic no
  longer has.
- E3: parts_sync.py keeps H2-H5's empty LCSC field (KiCad 10 field parity).
- cpl_check.py rewritten as a gate: places JLC's own footprint where the
  CPL says, every JLC pad must land on our pads (pegs included), pin n on
  our pin n wherever the pattern also fits at another turn; only
  non-polar two-pad parts may sit 180 deg round. 177/181 pass, 0 to fix.
- production.sh: Fabrication Toolkit CLI, then the gate; deletes the
  order zip if it fails. production/ regenerated through it.

3D / STEP: EasyEDA STEP models placed onto their pads (J1 M.2, J16, K5/K6,
U1/U9, SW2), LCSC STEPs for the KF250 terminals and fuses, standoffs
converted from VRML (wrl2step.py); review/MES4_Carrier_EC.step.

Enclosure: two-part FDM box generated from the board (FreeCAD): M3
heat-set inserts, connector openings, LED light guides and labels, M5
side tabs, engraved logo, P1S tolerances, no supports. The 82 MB
assembly STEP is regenerated, not committed.

Co-Authored-By: Claude Opus 5.5 <noreply@anthropic.com>
Parts:
- F3, F4: footprint Fuse:Fuse_2920_7451Metric -> MES4-Carrier-EC:Fuse_2920_7451Metric
Changed lines of the file:
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@@
 			(effects (font (size 1.27 1.27)))
 		)
-		(property "Footprint" "Fuse:Fuse_2920_7451Metric"
+		(property "Footprint" "MES4-Carrier-EC:Fuse_2920_7451Metric"
 			(at 185.42 58.42 0)
 			(effects (font (size 1.27 1.27)) (hide yes))
@@
 			(effects (font (size 1.27 1.27)))
 		)
-		(property "Footprint" "Fuse:Fuse_2920_7451Metric"
+		(property "Footprint" "MES4-Carrier-EC:Fuse_2920_7451Metric"
 			(at 185.42 162.56 0)
 			(effects (font (size 1.27 1.27)) (hide yes))
