File: MES4_Carrier_EC/Relays34.kicad_sch (KiCad schematic)
At the start: 34 parts, among them J8 RLY3 OUT, J9 RLY4 OUT, K3 SRD-5VDC-SL-A, K4 SRD-5VDC-SL-A, Q4 AO3400A, Q5 AO3400A, U4 TCA9535PWR, U5 INA226, U6 INA226

Commit message: Put relay coil feedback back on PA0-PA3 (MES4 GPIO standard)
All 14 module GPIOs now follow the MES4-CIF §2c table. The TCA9535 is
removed from the Relays 3-4 sheet and J1 fingers 43/45/47/49 drive the
relay 1-4 feedback dividers again. The winch relays are left undriven
(gate inputs no-connected, 100k pull-downs hold them off) until they
move to the TCA9535 + photoMOS design (HANDOFF.md step 2).

Removing U4 renumbers U5-U12 to U4-U11 and C15-C45 to C14-C44; the
README refs follow. Adds generator/checks.py (pin/pad, single-pin nets,
duplicate UUIDs, LCSC numbers), run by run.sh after ERC.

Co-Authored-By: Claude Opus 5.5 <noreply@anthropic.com>
Parts:
- removed C18: 100nF, Capacitor_SMD:C_0402_1005Metric, symbol Device:C
- removed D16, D17: SS34, Diode_SMD:D_SMA, symbol Device:D_Schottky
- removed R22, R27: 15k, Resistor_SMD:R_0402_1005Metric, symbol Device:R
- removed R23, R28: 100Ω, Resistor_SMD:R_0402_1005Metric, symbol Device:R
- removed U4: TCA9535PWR, Package_SO:TSSOP-24_4.4x7.8mm_P0.65mm, symbol MES4-Carrier-EC:TCA9535PWR
- removed U5, U6: INA226, Package_SO:VSSOP-10_3x3mm_P0.5mm, symbol Sensor_Energy:INA226
- added J8: RLY3 OUT, MES4-Carrier-EC:CONN-TH_KF250NH-3.5-2P, symbol Connector:Screw_Terminal_01x02
- added J9: RLY4 OUT, MES4-Carrier-EC:CONN-TH_KF250NH-3.5-2P, symbol Connector:Screw_Terminal_01x02
- added Q4, Q5: AO3400A, Package_TO_SOT_SMD:SOT-23, symbol Transistor_FET:AO3400A
- added R20, R25: 30mΩ, Resistor_SMD:R_1206_3216Metric, symbol Device:R
- added R24, R29: 100k, Resistor_SMD:R_0402_1005Metric, symbol Device:R
- C14: value 100nF -> 10nF; LCSC C1525 -> C15195
- C16: value 10nF -> 100nF; LCSC C15195 -> C1525
- D16: renamed from J8; value RLY3 OUT -> SS34; footprint MES4-Carrier-EC:CONN-TH_KF250NH-3.5-2P -> Diode_SMD:D_SMA; symbol Connector:Screw_Terminal_01x02 -> Device:D_Schottky; LCSC C976556 -> C8678
- D17: renamed from J9; value RLY4 OUT -> SS34; footprint MES4-Carrier-EC:CONN-TH_KF250NH-3.5-2P -> Diode_SMD:D_SMA; symbol Connector:Screw_Terminal_01x02 -> Device:D_Schottky; LCSC C976556 -> C8678
- R21: renamed from R24; value 100k -> 10k; LCSC C25741 -> C25744
- R22: renamed from R21; value 10k -> 15k; LCSC C25744 -> C25756
- R23: renamed from Q4; value AO3400A -> 100Ω; footprint Package_TO_SOT_SMD:SOT-23 -> Resistor_SMD:R_0402_1005Metric; symbol Transistor_FET:AO3400A -> Device:R; LCSC C20917 -> C25076
- R26: renamed from R29; value 100k -> 10k; LCSC C25741 -> C25744
- R27: renamed from R26; value 10k -> 15k; LCSC C25744 -> C25756
- R28: renamed from Q5; value AO3400A -> 100Ω; footprint Package_TO_SOT_SMD:SOT-23 -> Resistor_SMD:R_0402_1005Metric; symbol Transistor_FET:AO3400A -> Device:R; LCSC C20917 -> C25076
- U4: renamed from R20; value 30mΩ -> INA226; footprint Resistor_SMD:R_1206_3216Metric -> Package_SO:VSSOP-10_3x3mm_P0.5mm; symbol Device:R -> Sensor_Energy:INA226; LCSC C5375399 -> C49851
- U5: renamed from R25; value 30mΩ -> INA226; footprint Resistor_SMD:R_1206_3216Metric -> Package_SO:VSSOP-10_3x3mm_P0.5mm; symbol Device:R -> Sensor_Energy:INA226; LCSC C5375399 -> C49851
Connections:
- net +24V: now also U4.10 (Vin+), U4.8 (Vbus), U5.10 (Vin+), U5.8 (Vbus), R20.2, R25.2; no longer U4.2, U5.2
- net +3V3_MOD: now also C16.1, U4.1 (A1), U4.6 (VS), U5.1 (A1), U5.2 (A0), U5.6 (VS); no longer C14.1
- net GND: now also R22.2, R27.2, U4.2 (A0), U4.7 (GND), U5.7 (GND), Q4.2 (S), Q5.2 (S), R24.2, R29.2; no longer R21.2, R23.2 (S), R26.2, R28.2 (S)
- net GND_24V: now also J8.2 (Pin_2), J9.2 (Pin_2)
- net I2C1_SCL: now also U4.5 (SCL), U5.5 (SCL)
- net I2C1_SDA: now also U4.4 (SDA), U5.4 (SDA)
- net PA15: now also U4.3 (~{Alert}), U5.3 (~{Alert})
- net PA7: now also R28.1
- net PB3: now also R23.1
- net RLY3_OUT: now also J8.1 (Pin_1)
- net RLY4_OUT: now also J9.1 (Pin_1)
- net at K3.1: now also U4.9 (Vin-), R20.1; no longer U4.1
- net at D14.2 (A), K3.2: now also R21.1, Q4.3 (D); no longer R22.1, R23.3 (D)
- net at K4.1: now also U5.9 (Vin-), R25.1; no longer U5.1
- net at R26.1: now also D15.2 (A), K4.2, Q5.3 (D); no longer R28.1 (G)
- net RLY3_FB renamed PA3
- net PA3: now also R26.2, R27.1; no longer R22.2
- removed net RLY4_FB: C16.1, R27.2
- new net: Q4.1 (G), R23.2, R24.1
- new net: Q5.1 (G), R28.2, R29.1
- new net PA2: C14.1, R21.2, R22.1
- no-connect marks 13 -> 0
Other:
- note added: "Coil feedback (PA2): HIGH (3.0 V) = coil off and intact, LOW = energised. INA226 0x44 (A1 = VS, A0 = GND): load current (30 mΩ, LSB 100 µA) + 24 V rail; ALERT → PA15. LED6: output ON; its 6.7 mA also lets the INA226 see the contact close with no load. F5: 3A hold PTC, so a shorted output trips only this channel. D16: load flyback. Q4 AO3400A: R23 100 Ω gate, R24 100k pull-down = OFF in reset (CIF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"
- note added: "Coil feedback (PA3): HIGH (3.0 V) = coil off and intact, LOW = energised. INA226 0x45 (A1 = VS, A0 = VS): load current (30 mΩ, LSB 100 µA) + 24 V rail; ALERT → PA15. LED7: output ON; its 6.7 mA also lets the INA226 see the contact close with no load. F6: 3A hold PTC, so a shorted output trips only this channel. D17: load flyback. Q5 AO3400A: R28 100 Ω gate, R29 100k pull-down = OFF in reset (CIF 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"
- note added: "Relay 3 (battery stopper): drive PB3, coil feedback PA2, INA226 U4 at 0x44"
- note added: "Relay 4 (spare): drive PA7, coil feedback PA3, INA226 U5 at 0x45"
- note removed: "Coil feedback (RLY3_FB, TCA9535 P02): HIGH (3.0 V) = coil off and intact, LOW = energised. INA226 0x44 (A1 = VS, A0 = GND): load current (30 mΩ, LSB 100 µA) + 24 V rail; ALERT → PA15. LED6: output ON; its 6.7 mA also lets the INA226 see the contact close with no load. F5: 3A hold PTC, so a shorted output trips only this channel. D16: load flyback. Q4 AO3400A: R23 100 Ω gate, R24 100k pull-down = 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"
- note removed: "Coil feedback (RLY4_FB, TCA9535 P03): HIGH (3.0 V) = coil off and intact, LOW = energised. INA226 0x45 (A1 = VS, A0 = VS): load current (30 mΩ, LSB 100 µA) + 24 V rail; ALERT → PA15. LED7: output ON; its 6.7 mA also lets the INA226 see the contact close with no load. F6: 3A hold PTC, so a shorted output trips only this channel. D17: load flyback. Q5 AO3400A: R28 100 Ω gate, R29 100k pull-down = O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"
- note removed: "Coil feedback expander (I²C1 0x20)"
- note removed: "Relay 3 (battery stopper): drive PB3, coil feedback RLY3_FB, INA226 U5 at 0x44"
- note removed: "Relay 4 (spare): drive PA7, coil feedback RLY4_FB, INA226 U6 at 0x45"
- note removed: "U4 TCA9535PWR: A2 / A1 / A0 = GND → I²C1 0x20 (no clash with the INA226s at 0x40-0x45). P00-P03 = relay 1-4 coil feedback (10k / 15k + 10 nF dividers, 3.0 V = coil off; inputs 5.5 V-tolerant). INT not connected: PA0 drives the winch, so poll the expander. P04-P17 spare (12 inputs for later): no internal pull-ups, so set them as outputs, LOW, at start-up. Read input port 0 (reg 0x00) ≥ 30 ms after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"
- moved on the sheet: R21, R22, R26, R27

Commit message: Drop relay coil feedback; winch on PA0/PA1, servo on USART2
User decision: free the four feedback pins instead of adding an I²C
expander. The Flasher template's 10k/15k/10 nF dividers are removed from
all relay channels and relay diagnosis is INA226-only. PA0/PA1 drive the
IM03GR winch relays again and PA2/PA3 carry the door servo UART
(USART2), so the SC16IS740 bridge, its crystal and caps, and the unused
TCA9535 code are removed. This deliberately differs from the MES4-CIF
§2c GPIO table; the GPIO map, root notes, README and HANDOFF say so.

189 parts, ERC clean, checks.py passes. README refs follow the
renumbering.

Co-Authored-By: Claude Opus 5.5 <noreply@anthropic.com>
Parts:
- removed C14, C15: 10nF, Capacitor_SMD:C_0402_1005Metric, symbol Device:C
- removed C16, C17: 100nF, Capacitor_SMD:C_0402_1005Metric, symbol Device:C
- removed F5, F6: 3A, Fuse:Fuse_2920_7451Metric, symbol Device:Polyfuse
- removed J8: RLY3 OUT, MES4-Carrier-EC:CONN-TH_KF250NH-3.5-2P, symbol Connector:Screw_Terminal_01x02
- removed J9: RLY4 OUT, MES4-Carrier-EC:CONN-TH_KF250NH-3.5-2P, symbol Connector:Screw_Terminal_01x02
- removed R24, R29: 100k, Resistor_SMD:R_0402_1005Metric, symbol Device:R
- removed R25: 30mΩ, Resistor_SMD:R_1206_3216Metric, symbol Device:R
- removed R26: 10k, Resistor_SMD:R_0402_1005Metric, symbol Device:R
- removed R27: 15k, Resistor_SMD:R_0402_1005Metric, symbol Device:R
- removed R28: 100Ω, Resistor_SMD:R_0402_1005Metric, symbol Device:R
- added C12, C13: 100nF, Capacitor_SMD:C_0402_1005Metric, symbol Device:C
- added LED6, LED7: Yellow, LED_SMD:LED_0805_2012Metric, symbol Device:LED
- added R16, R19: 30mΩ, Resistor_SMD:R_1206_3216Metric, symbol Device:R
- added R17: 100Ω, Resistor_SMD:R_0402_1005Metric, symbol Device:R
- added R18: 100k, Resistor_SMD:R_0402_1005Metric, symbol Device:R
- F5: renamed from R30; value 3.3k -> 3A; footprint Resistor_SMD:R_1206_3216Metric -> Fuse:Fuse_2920_7451Metric; symbol Device:R -> Device:Polyfuse; LCSC C26032 -> C22435908
- F6: renamed from R31; value 3.3k -> 3A; footprint Resistor_SMD:R_1206_3216Metric -> Fuse:Fuse_2920_7451Metric; symbol Device:R -> Device:Polyfuse; LCSC C26032 -> C22435908
- J8: renamed from LED6; value Yellow -> RLY3 OUT; footprint LED_SMD:LED_0805_2012Metric -> MES4-Carrier-EC:CONN-TH_KF250NH-3.5-2P; symbol Device:LED -> Connector:Screw_Terminal_01x02; LCSC C2296 -> C976556
- J9: renamed from LED7; value Yellow -> RLY4 OUT; footprint LED_SMD:LED_0805_2012Metric -> MES4-Carrier-EC:CONN-TH_KF250NH-3.5-2P; symbol Device:LED -> Connector:Screw_Terminal_01x02; LCSC C2296 -> C976556
- R20: value 30mΩ -> 100Ω; footprint Resistor_SMD:R_1206_3216Metric -> Resistor_SMD:R_0402_1005Metric; LCSC C5375399 -> C25076
- R21: value 10k -> 100k; LCSC C25744 -> C25741
- R22: value 15k -> 3.3k; footprint Resistor_SMD:R_0402_1005Metric -> Resistor_SMD:R_1206_3216Metric; LCSC C25756 -> C26032
- R23: value 100Ω -> 3.3k; footprint Resistor_SMD:R_0402_1005Metric -> Resistor_SMD:R_1206_3216Metric; LCSC C25076 -> C26032
Connections:
- net +24V: now also R16.2, R19.2; no longer R20.2
- net +3V3_MOD: now also C12.1, C13.1
- net GND: now also R21.2, C12.2, C13.2, R18.2; no longer R22.2
- net GND_24V: now also J8.2 (Pin_2), J9.2 (Pin_2), LED6.1 (K), LED7.1 (K); no longer J8.1 (K), J9.1 (K)
- net PA7: now also R20.1
- net PB3: now also R17.1; no longer R23.1
- net RLY3_OUT: now also F5.2, J8.1 (Pin_1), R22.1; no longer F5.1
- net RLY4_OUT: now also F6.2, J9.1 (Pin_1), R23.1; no longer F6.1
- net at R23.2: now also LED7.2 (A); no longer Q4.1 (G)
- net at D14.2 (A), K3.2, Q4.3 (D): no longer R21.1
- net at Q5.1 (G): now also R20.2, R21.1
- net at K3.1, U4.9 (Vin-): now also R16.1; no longer R20.1
- net at K4.1, U5.9 (Vin-): now also R19.1
- net at K3.3: now also F5.1
- net at K4.3: now also F6.1
- removed net PA2: R21.2, R22.1
- new net: Q4.1 (G), R17.2, R18.1
- new net: LED6.2 (A), R22.2
Other:
- note added: "No coil feedback: PA0-PA3 drive the winch and the servo UART; the INA226 does the diagnosis. INA226 0x44 (A1 = VS, A0 = GND): load current (30 mΩ, LSB 100 µA) + 24 V rail; ALERT → PA15. LED6: output ON; its 6.7 mA also lets the INA226 see the contact close with no load. F5: 3A hold PTC, so a shorted output trips only this channel. D16: load flyback. Q4 AO3400A: R17 100 Ω gate, R18 100k pull-down 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"
- note added: "No coil feedback: PA0-PA3 drive the winch and the servo UART; the INA226 does the diagnosis. INA226 0x45 (A1 = VS, A0 = VS): load current (30 mΩ, LSB 100 µA) + 24 V rail; ALERT → PA15. LED7: output ON; its 6.7 mA also lets the INA226 see the contact close with no load. F6: 3A hold PTC, so a shorted output trips only this channel. D17: load flyback. Q5 AO3400A: R20 100 Ω gate, R21 100k pull-down =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"
- note added: "Relay 3 (battery stopper): drive PB3, INA226 U4 at 0x44"
- note added: "Relay 4 (spare): drive PA7, INA226 U5 at 0x45"
- note removed: "Coil feedback (PA2): HIGH (3.0 V) = coil off and intact, LOW = energised. INA226 0x44 (A1 = VS, A0 = GND): load current (30 mΩ, LSB 100 µA) + 24 V rail; ALERT → PA15. LED6: output ON; its 6.7 mA also lets the INA226 see the contact close with no load. F5: 3A hold PTC, so a shorted output trips only this channel. D16: load flyback. Q4 AO3400A: R23 100 Ω gate, R24 100k pull-down = OFF in reset (CIF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"
- note removed: "Coil feedback (PA3): HIGH (3.0 V) = coil off and intact, LOW = energised. INA226 0x45 (A1 = VS, A0 = VS): load current (30 mΩ, LSB 100 µA) + 24 V rail; ALERT → PA15. LED7: output ON; its 6.7 mA also lets the INA226 see the contact close with no load. F6: 3A hold PTC, so a shorted output trips only this channel. D17: load flyback. Q5 AO3400A: R28 100 Ω gate, R29 100k pull-down = OFF in reset (CIF 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"
- note removed: "Relay 3 (battery stopper): drive PB3, coil feedback PA2, INA226 U4 at 0x44"
- note removed: "Relay 4 (spare): drive PA7, coil feedback PA3, INA226 U5 at 0x45"

Commit message: Address design review R1: INA236, J15 polarity, review fixes
M1: U2-U5 are now TI INA236AIDDFR (C5443912, 50 V abs max, TSOT-23-8)
instead of the INA226 (40 V), since the SMBJ30A clamps at up to 48.4 V.
A project INA236 symbol keeps the INA226 body so the Flasher relay
wiring lands on the same pins; A1 and VBUS are gone (bus read on IN-),
addresses 0x40-0x43 via A0 = GND / VS / SDA / SCL. Same CONFIG / CAL /
MASK / ALERT values; notes give the 1.6 mV bus LSB and Device ID.
M3: J15 servo 24 V is pin 1 = +24 V like every power terminal.
L4: R38 servo RX series resistor 1k (limits PA3 back-feed).
L2: "current present" threshold 3 mA. L6: Power notes use 13 A / 2.2 W.
M2 / L5: silkscreen notes for "5V LOAD CELL - NEVER 24V" and
"CAN - NOT ETHERNET" (no keyed connector, by choice).
RJ45 1x4 footprint rebuilt from the HCTL drawing (14.0 mm ports,
Ø1.5 shield and Ø3.2 peg positions); U1 / U9 / U10 checked against the
JLC library and YLPTEC drawing. HANDOFF gains the review status table
and a layout checklist.

Co-Authored-By: Claude Opus 5.5 <noreply@anthropic.com>
Parts:
- removed D16, D17: SS34, Diode_SMD:D_SMA, symbol Device:D_Schottky
- removed U4, U5: INA226, Package_SO:VSSOP-10_3x3mm_P0.5mm, symbol Sensor_Energy:INA226
- added LED6, LED7: Yellow, LED_SMD:LED_0805_2012Metric, symbol Device:LED
- added U4, U5: INA236, Package_TO_SOT_SMD:TSOT-23-8, symbol MES4-Carrier-EC:INA236
- D16: renamed from LED6; value Yellow -> SS34; footprint LED_SMD:LED_0805_2012Metric -> Diode_SMD:D_SMA; symbol Device:LED -> Device:D_Schottky; LCSC C2296 -> C8678
- D17: renamed from LED7; value Yellow -> SS34; footprint LED_SMD:LED_0805_2012Metric -> Diode_SMD:D_SMA; symbol Device:LED -> Device:D_Schottky; LCSC C2296 -> C8678
Connections:
- net +24V: now also U4.1 (IN+), U5.1 (IN+)
- net +3V3_MOD: now also U4.4 (VS), U5.4 (VS)
- net GND: now also U4.3 (GND), U5.3 (GND)
- net GND_24V: now also D16.2 (A), D17.2 (A), LED6.1 (K), LED7.1 (K); no longer D16.1 (K), D17.1 (K)
- net I2C1_SCL: now also U4.5 (SCL), U5.5 (SCL), U5.7 (A0)
- net I2C1_SDA: now also U4.6 (SDA), U4.7 (A0), U5.6 (SDA)
- net PA15: now also U4.8 (~{ALERT}), U5.8 (~{ALERT})
- net RLY3_OUT: now also D16.1 (K)
- net RLY4_OUT: now also D17.1 (K)
- net at R23.2: now also LED7.2 (A); no longer D17.2 (A)
- net at R22.2: now also LED6.2 (A); no longer D16.2 (A)
- net at K3.1, R16.1: now also U4.2 (IN-)
- net at K4.1, R19.1: now also U5.2 (IN-)
Other:
- note added: "No coil feedback: PA0-PA3 drive the winch and the servo UART; the INA236 does the diagnosis. INA236 0x42 (A0 = SDA): load current (30 mΩ, LSB 100 µA) + 24 V rail (read on IN-); ALERT → PA15. LED6: output ON; its 6.7 mA also lets the INA236 see the contact close with no load. F5: 3A hold PTC, so a shorted output trips only this channel. D16: load flyback. Q4 AO3400A: R17 100 Ω gate, R18 100k pull-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"
- note added: "No coil feedback: PA0-PA3 drive the winch and the servo UART; the INA236 does the diagnosis. INA236 0x43 (A0 = SCL): load current (30 mΩ, LSB 100 µA) + 24 V rail (read on IN-); ALERT → PA15. LED7: output ON; its 6.7 mA also lets the INA236 see the contact close with no load. F6: 3A hold PTC, so a shorted output trips only this channel. D17: load flyback. Q5 AO3400A: R20 100 Ω gate, R21 100k pull-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"
- note added: "Relay 3 (battery stopper): drive PB3, INA236 U4 at 0x42"
- note added: "Relay 4 (spare): drive PA7, INA236 U5 at 0x43"
- note removed: "No coil feedback: PA0-PA3 drive the winch and the servo UART; the INA226 does the diagnosis. INA226 0x44 (A1 = VS, A0 = GND): load current (30 mΩ, LSB 100 µA) + 24 V rail; ALERT → PA15. LED6: output ON; its 6.7 mA also lets the INA226 see the contact close with no load. F5: 3A hold PTC, so a shorted output trips only this channel. D16: load flyback. Q4 AO3400A: R17 100 Ω gate, R18 100k pull-down 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"
- note removed: "No coil feedback: PA0-PA3 drive the winch and the servo UART; the INA226 does the diagnosis. INA226 0x45 (A1 = VS, A0 = VS): load current (30 mΩ, LSB 100 µA) + 24 V rail; ALERT → PA15. LED7: output ON; its 6.7 mA also lets the INA226 see the contact close with no load. F6: 3A hold PTC, so a shorted output trips only this channel. D17: load flyback. Q5 AO3400A: R20 100 Ω gate, R21 100k pull-down =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"
- note removed: "Relay 3 (battery stopper): drive PB3, INA226 U4 at 0x44"
- note removed: "Relay 4 (spare): drive PA7, INA226 U5 at 0x45"

Commit message: Import all footprints into the PCB; TI land pattern for the INA236
MES4_Carrier_EC.kicad_pcb: all 190 footprints and 146 nets, grouped by
schematic sheet below the 200 x 100 mm outline, ready to place. Each
footprint carries its symbol path (F8 updates it instead of duplicating),
nets, LCSC number and BOM setting. DRC: schematic parity 0 issues,
0 clearance errors; 450 unconnected items (unrouted).

generator/import_footprints.py does the one-time import with KiCad's
pcbnew Python and refuses a board that already has footprints.

U2-U5 INA236 now use the project footprint TSOT-23-8_TI_DDF (TI DDF0008A
land pattern: 1.05 x 0.45 mm pads, rows 2.6 mm apart). KiCad's generic
TSOT-23-8 left 0.15 mm pad gaps against the 0.2 mm clearance.

.kicad_pro regenerated: KiCad had rewritten it on exit and dropped the
Winch_48V net class. HANDOFF notes the import, the footprint and the fix.

Co-Authored-By: Claude Opus 5.5 <noreply@anthropic.com>
Parts:
- U4, U5: footprint Package_TO_SOT_SMD:TSOT-23-8 -> MES4-Carrier-EC:TSOT-23-8_TI_DDF
Changed lines of the file:
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@@
 			(effects (font (size 1.27 1.27)) (justify left))
 		)
-		(property "Footprint" "Package_TO_SOT_SMD:TSOT-23-8"
+		(property "Footprint" "MES4-Carrier-EC:TSOT-23-8_TI_DDF"
 			(at 226.06 96.52 0)
 			(effects (font (size 1.27 1.27)) (hide yes))
@@
 			(effects (font (size 1.27 1.27)) (justify left))
 		)
-		(property "Footprint" "Package_TO_SOT_SMD:TSOT-23-8"
+		(property "Footprint" "MES4-Carrier-EC:TSOT-23-8_TI_DDF"
 			(at 226.06 200.66 0)
 			(effects (font (size 1.27 1.27)) (hide yes))

Commit message: One ground and a 4-layer board
- GND_24V merged into GND (ONE_GND in gen.py): every GND_24V power symbol
  becomes GND, net tie NT1 left out, notes reworded. Symbol UUIDs unchanged,
  so every footprint keeps its link.
- 4 layers, JLC04161H-7628 stackup (1.6 mm, ENIG): Top Signal / GND plane
  (In1) / +24V plane (In2) / Bottom Signal.
- Net classes: Out_3A (1.5 mm) for +24V_SRV, +5V_SCR, VBUS_SCR; +24V_AUX to
  24V_Power; +5V_SRV, +9V_IMU, IMU_9V to Power; INA236 shunt pattern fixed
  (Net-(U*-IN-)).
- J1's NPTH holes back to F&B.Cu as in its library footprint.

ERC 0, checks passed, DRC 11 silkscreen warnings, schematic parity clean.

Co-Authored-By: Claude Opus 5.5 <noreply@anthropic.com>
Connections:
- net GND_24V is gone; now on net GND: D16.2 (A), D17.2 (A), J8.2 (Pin_2), J9.2 (Pin_2), LED6.1 (K), LED7.1 (K)

Commit message: Check CPL rotations against JLC's footprints; fix Q1, K1-K4, J5
- cpl_check.py: fetches each LCSC part's EasyEDA footprint, matches
  pads (polarity names, numbers or shape), fits the rotation / offset
  JLC needs and compares with production/positions.csv.
- Q1 (TO-252) needs +180 deg and -1.8 mm, K1-K4 (SRD relays) +180 deg,
  J5 (XT30) +9.7 mm: set as Fabrication Toolkit FT Rotation / Position
  Offset fields on the symbols (gen.py, parts.py), copied to the board
  by parts_sync.py.
- production/ regenerated with the toolkit CLI: 169 of 181 placements
  match JLC; C1 / C5 / C27 (no JLC footprint) to check in the preview.
- HANDOFF updated.

Co-Authored-By: Claude Opus 5.5 <noreply@anthropic.com>
Parts:
- K3, K4: FT Rotation Offset (none) -> 180
Changed lines of the file:
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@@
+			(effects (font (size 1.27 1.27)) (hide yes))
+		)
+		(property "FT Rotation Offset" "180"
+			(at 172.72 66.04 0)
 			(effects (font (size 1.27 1.27)) (hide yes))
 		)
@@
 			(at 172.72 170.18 0)
 			(effects (font (size 1.27 1.27)) (hide yes))
+		)
+		(property "FT Rotation Offset" "180"
+			(at 172.72 170.18 0)
+			(effects (font (size 1.27 1.27)) (hide yes))
